Commit message: 增加了启动脚本，当前支持启动宇树go1、a1，合作机械臂，傅里叶智能gr1,

File: simulation_all/src/robots/gh1_description/urdf/gh1_description.urdf (robot description, URDF)
Before this commit: robot gh1_description, 20 links, 19 joints
Links:
- added link imu_link; visual box size=0.05 0.05 0.02
- link Left_ankle_pitch_Link: geometry collision box size=0.25 0.07 0.015; visual mesh filename=package://gh1_description/meshes/Left_ankle_pitch_Link.STL
- link Left_elbow_pitch_Link: geometry collision cylinder length=0.01 radius=0.032; visual mesh filename=package://gh1_description/meshes/Left_elbow_pitch_Link.STL
- link Left_hip_pitch_Link: geometry collision cylinder length=0.32 radius=0.04; visual mesh filename=package://gh1_description/meshes/Left_hip_pitch_Link.STL
- link Left_hip_roll_Link: geometry collision cylinder length=0.01 radius=0.02; visual mesh filename=package://gh1_description/meshes/Left_hip_roll_Link.STL
- link Left_hip_yaw_Link: geometry collision cylinder length=0.01 radius=0.02; visual mesh filename=package://gh1_description/meshes/Left_hip_yaw_Link.STL
- link Left_knee_Link: geometry collision cylinder length=0.3 radius=0.02; visual mesh filename=package://gh1_description/meshes/Left_knee_Link.STL
- link Left_shoulder_pitch_Link: geometry collision cylinder length=0.0372 radius=0.05; visual mesh filename=package://gh1_description/meshes/Left_shoulder_pitch_Link.S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
- link Left_shoulder_roll_Link: geometry collision cylinder length=0.05 radius=0.049; visual mesh filename=package://gh1_description/meshes/Left_shoulder_roll_Link.STL
- link Left_shoulder_yaw_Link: geometry collision cylinder length=0.1 radius=0.02; visual mesh filename=package://gh1_description/meshes/Left_shoulder_yaw_Link.STL
- link Right_ankle_pitch_Link: geometry collision box size=0.25 0.07 0.015; visual mesh filename=package://gh1_description/meshes/Right_ankle_pitch_Link.STL
- link Right_elbow_pitch_Link: geometry collision cylinder length=0.01 radius=0.032; visual mesh filename=package://gh1_description/meshes/Right_elbow_pitch_Link.STL
- link Right_hip_pitch_Link: geometry collision cylinder length=0.32 radius=0.04; visual mesh filename=package://gh1_description/meshes/Right_hip_pitch_Link.STL
- link Right_hip_roll_Link: geometry collision cylinder length=0.01 radius=0.02; visual mesh filename=package://gh1_description/meshes/Right_hip_roll_Link.STL
- link Right_hip_yaw_Link: geometry collision cylinder length=0.01 radius=0.02; visual mesh filename=package://gh1_description/meshes/Right_hip_yaw_Link.STL
- link Right_knee_Link: geometry collision cylinder length=0.3 radius=0.02; visual mesh filename=package://gh1_description/meshes/Right_knee_Link.STL
- link Right_shoulder_pitch_Link: geometry collision cylinder length=0.0372 radius=0.05; visual mesh filename=package://gh1_description/meshes/Right_shoulder_pitch_Link.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
- link Right_shoulder_roll_Link: geometry collision cylinder length=0.05 radius=0.049; visual mesh filename=package://gh1_description/meshes/Right_shoulder_roll_Link.S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
- link Right_shoulder_yaw_Link: geometry collision cylinder length=0.1 radius=0.02; visual mesh filename=package://gh1_description/meshes/Right_shoulder_yaw_Link.STL
- link body: geometry collision box size=0.130 0.3 0.35; visual mesh filename=package://gh1_description/meshes/body.STL
Joints:
- added joint z_joint_imu: type fixed, parent body, child imu_link, origin xyz=-0.0648 0 -0.1015 rpy=0 0 0

File: simulation_all/src/robots/go1_description/xacro/robot.xacro (robot description, xacro)
@@ -2,124 +2,126 @@
 <robot name="go1"
     xmlns:xacro="http://www.ros.org/wiki/xacro">
-    <xacro:arg name="DEBUG" default="false"/>
-    <xacro:include filename="$(find go1_description)/xacro/const.xacro"/>
-    <xacro:include filename="$(find go1_description)/xacro/materials.xacro"/>
-    <xacro:include filename="$(find go1_description)/xacro/leg.xacro"/>
+    <xacro:arg name="DEBUG" default="false" />
+    <xacro:include filename="$(find go1_description)/xacro/const.xacro" />
+    <xacro:include filename="$(find go1_description)/xacro/materials.xacro" />
+    <xacro:include filename="$(find go1_description)/xacro/leg.xacro" />
     <!-- <xacro:include filename="$(find go1_description)/xacro/stairs.xacro"/> -->
-    <xacro:include filename="$(find go1_description)/xacro/gazebo.xacro"/>
-    <xacro:include filename="$(find go1_description)/xacro/depthCamera.xacro"/>
-    <xacro:include filename="$(find go1_description)/xacro/ultraSound.xacro"/>
+    <xacro:include filename="$(find go1_description)/xacro/gazebo.xacro" />
+    <xacro:include filename="$(find go1_description)/xacro/depthCamera.xacro" />
+    <xacro:include filename="$(find go1_description)/xacro/ultraSound.xacro" />
     <!-- <xacro:include filename="$(find go1_gazebo)/launch/stairs.urdf.xacro"/> -->
     <!-- <xacro:stairs stairs="15" xpos="0" ypos="0" zpos="0" /> -->
     <!-- Rotor related joint and link is only for demonstrate location. -->
-    <!-- Actually, the rotor will rotate and the joint is not fixed. Reduction ratio should be considered. -->
+    <!-- Actually, the rotor will rotate and the joint is not fixed. Reduction ratio should be
+    considered. -->
     <!-- Debug mode will hung up the robot, use "true" or "false" to switch it. -->
     <xacro:if value="$(arg DEBUG)">
-        <link name="world"/>
+        <link name="world" />
         <joint name="base_static_joint" type="fixed">
-            <origin rpy="0 0 0" xyz="0 0 0"/>
-            <parent link="world"/>
-            <child link="base"/>
+            <origin rpy="0 0 0" xyz="0 0 0" />
+            <parent link="world" />
+            <child link="base" />
         </joint>
     </xacro:if>
     <link name="base">
         <visual>
-            <origin rpy="0 0 0" xyz="0 0 0"/>
+            <origin rpy="0 0 0" xyz="0 0 0" />
             <geometry>
-                <box size="0.001 0.001 0.001"/>
+                <box size="0.001 0.001 0.001" />
             </geometry>
         </visual>
     </link>
     <joint name="floating_base" type="fixed">
-        <origin rpy="0 0 0" xyz="0 0 0"/>
-        <parent link="base"/>
-        <child link="trunk"/>
+        <origin rpy="0 0 0" xyz="0 0 0" />
+        <parent link="base" />
+        <child link="trunk" />
     </joint>
     <link name="trunk">
         <visual>
-            <origin rpy="0 0 0" xyz="0 0 0"/>
+            <origin rpy="0 0 0" xyz="0 0 0" />
             <geometry>
-                <mesh filename="package://go1_description/meshes/trunk.dae" scale="1 1 1"/>
+                <mesh filename="package://go1_description/meshes/trunk.dae" scale="1 1 1" />
             </geometry>
             <!-- <material name="orange"/> -->
         </visual>
         <collision>
-            <origin rpy="0 0 0" xyz="0 0 0"/>
+            <origin rpy="0 0 0" xyz="0 0 0" />
             <geometry>
-                <box size="${trunk_length} ${trunk_width} ${trunk_height}"/>
+                <box size="${trunk_length} ${trunk_width} ${trunk_height}" />
             </geometry>
         </collision>
         <inertial>
-            <origin rpy="0 0 0" xyz="${trunk_com_x} ${trunk_com_y} ${trunk_com_z}"/>
-            <mass value="${trunk_mass}"/>
-            <inertia ixx="${trunk_ixx}" ixy="${trunk_ixy}" ixz="${trunk_ixz}" iyy="${trunk_iyy}" iyz="${trunk_iyz}" izz="${trunk_izz}"/>
+            <origin rpy="0 0 0" xyz="${trunk_com_x} ${trunk_com_y} ${trunk_com_z}" />
+            <mass value="${trunk_mass}" />
+            <inertia ixx="${trunk_ixx}" ixy="${trunk_ixy}" ixz="${trunk_ixz}" iyy="${trunk_iyy}"
+                iyz="${trunk_iyz}" izz="${trunk_izz}" />
         </inertial>
     </link>
     <joint name="imu_joint" type="fixed">
-        <parent link="trunk"/>
-        <child link="imu_link"/>
-        <origin rpy="0 0 0" xyz="-0.01592 -0.06659 -0.00617"/>
+        <parent link="trunk" />
+        <child link="imu_link" />
+        <origin rpy="0 0 0" xyz="-0.01592 -0.06659 -0.00617" />
     </joint>
     <link name="imu_link">
         <inertial>
-            <mass value="0.001"/>
-            <origin rpy="0 0 0" xyz="0 0 0"/>
-            <inertia ixx="0.0001" ixy="0" ixz="0" iyy="0.0001" iyz="0" izz="0.0001"/>
+            <mass value="0.001" />
+            <origin rpy="0 0 0" xyz="0 0 0" />
+            <inertia ixx="0.0001" ixy="0" ixz="0" iyy="0.0001" iyz="0" izz="0.0001" />
         </inertial>
         <visual>
-            <origin rpy="0 0 0" xyz="0 0 0"/>
+            <origin rpy="0 0 0" xyz="0 0 0" />
             <geometry>
-                <box size="0.001 0.001 0.001"/>
+                <box size="0.001 0.001 0.001" />
             </geometry>
             <!-- <material name="red"/> -->
         </visual>
         <collision>
-            <origin rpy="0 0 0" xyz="0 0 0"/>
+            <origin rpy="0 0 0" xyz="0 0 0" />
             <geometry>
-                <box size=".001 .001 .001"/>
+                <box size=".001 .001 .001" />
             </geometry>
         </collision>
     </link>
-    <xacro:leg name="FR" mirror="-1" mirror_dae= "False" front_hind="1" front_hind_dae="True" />
+    <xacro:leg name="FR" mirror="-1" mirror_dae="False" front_hind="1" front_hind_dae="True" />
     <xacro:leg name="FL" mirror="1" mirror_dae="True" front_hind="1" front_hind_dae="True" />
     <xacro:leg name="RR" mirror="-1" mirror_dae="False" front_hind="-1" front_hind_dae="False" />
     <xacro:leg name="RL" mirror="1" mirror_dae="True" front_hind="-1" front_hind_dae="False" />
     <xacro:depthCamera camID="1" name="face">
-        <origin rpy="${PI} 0 0" xyz="0.2785 0.0125 0.0167"/>
+        <origin rpy="${PI} 0 0" xyz="0.2785 0.0125 0.0167" />
     </xacro:depthCamera>
     <xacro:depthCamera camID="2" name="chin">
-        <origin rpy="${PI} ${PI/2} 0" xyz="0.2522 0.0125 -0.0436"/>
+        <origin rpy="${PI} ${PI/2} 0" xyz="0.2522 0.0125 -0.0436" />
     </xacro:depthCamera>
     <xacro:depthCamera camID="3" name="left">
-        <origin rpy="${PI} 0.2618 ${PI/2}" xyz="-0.066 0.082 -0.0176"/>
+        <origin rpy="${PI} 0.2618 ${PI/2}" xyz="-0.066 0.082 -0.0176" />
     </xacro:depthCamera>
     <xacro:depthCamera camID="4" name="right">
-        <origin rpy="${PI} 0.2618 ${-PI/2}" xyz="-0.041 -0.082 -0.0176"/>
+        <origin rpy="${PI} 0.2618 ${-PI/2}" xyz="-0.041 -0.082 -0.0176" />
     </xacro:depthCamera>
     <xacro:depthCamera camID="5" name="rearDown">
-        <origin rpy="${PI} ${PI/2} 0" xyz="-0.0825 0.0125 -0.04365"/>
+        <origin rpy="${PI} ${PI/2} 0" xyz="-0.0825 0.0125 -0.04365" />
     </xacro:depthCamera>
     <joint name="camera_laserscan_joint_left" type="fixed">
-        <origin rpy="0 0.2618 0" xyz="0 0 0"/>
-        <parent link="camera_left"/>
-        <child link="camera_laserscan_link_left"/>
+        <origin rpy="0 0.2618 0" xyz="0 0 0" />
+        <parent link="camera_left" />
+        <child link="camera_laserscan_link_left" />
     </joint>
     <link name="camera_laserscan_link_left">
     </link>
     <joint name="camera_laserscan_joint_right" type="fixed">
-        <origin rpy="0 0.2618 0" xyz="0 0 0"/>
-        <parent link="camera_right"/>
-        <child link="camera_laserscan_link_right"/>
+        <origin rpy="0 0.2618 0" xyz="0 0 0" />
+        <parent link="camera_right" />
+        <child link="camera_laserscan_link_right" />
     </joint>
     <link name="camera_laserscan_link_right">
     </link>
     <xacro:ultraSound name="left">
-        <origin rpy="0 0.2618 ${PI/2}" xyz="-0.0535  0.0826 0.00868"/>
+        <origin rpy="0 0.2618 ${PI/2}" xyz="-0.0535  0.0826 0.00868" />
     </xacro:ultraSound>
     <xacro:ultraSound name="right">
-        <origin rpy="0 0.2618 ${-PI/2}" xyz="-0.0535 -0.0826 0.00868"/>
+        <origin rpy="0 0.2618 ${-PI/2}" xyz="-0.0535 -0.0826 0.00868" />
     </xacro:ultraSound>
     <xacro:ultraSound name="face">
-        <origin rpy="0 0 0" xyz="0.2747 0.0 -0.0088"/>
+        <origin rpy="0 0 0" xyz="0.2747 0.0 -0.0088" />
     </xacro:ultraSound>
 </robot>

File: simulation_all/src/robots/iris_description/urdf/iris3.urdf (robot description, URDF)
Before this commit: robot iris3, 8 links, 7 joints
Links:
- link Link1: geometry collision mesh filename=package://iris_description/meshes/Link1.STL; visual mesh filename=package://iris_description/meshes/Link1.STL
- link Link2: geometry collision mesh filename=package://iris_description/meshes/Link2.STL; visual mesh filename=package://iris_description/meshes/Link2.STL
- link Link3: geometry collision mesh filename=package://iris_description/meshes/Link3.STL; visual mesh filename=package://iris_description/meshes/Link3.STL
- link Link4: geometry collision mesh filename=package://iris_description/meshes/Link4.STL; visual mesh filename=package://iris_description/meshes/Link4.STL
- link Link5: geometry collision mesh filename=package://iris_description/meshes/Link5.STL; visual mesh filename=package://iris_description/meshes/Link5.STL
- link Link6: geometry collision mesh filename=package://iris_description/meshes/Link6.STL; visual mesh filename=package://iris_description/meshes/Link6.STL
- link base_link: geometry collision mesh filename=package://iris_description/meshes/base_link.STL; visual mesh filename=package://iris_description/meshes/base_link.STL
