Commit message: 添加mz机器人模型

File: src/robots/mz_description/urdf/mz_description.urdf (robot description, URDF)
Before this commit: robot mz_description, 18 links, 17 joints
Links:
- removed link FL_FOOT
- removed link FR_FOOT
- removed link RL_FOOT
- removed link RR_FOOT
- added link FL_foot, mass 0.07; collision sphere radius=0.0235; visual sphere radius=0.015
- added link FL_thigh_shoulder
- added link FR_foot, mass 0.07; collision sphere radius=0.0235; visual sphere radius=0.01
- added link FR_thigh_shoulder
- added link RL_foot, mass 0.07; collision sphere radius=0.0235; visual sphere radius=0.01
- added link RL_thigh_shoulder
- added link RR_foot, mass 0.07; collision sphere radius=0.0235; visual sphere radius=0.01
- added link RR_thigh_shoulder
- added link imu_link, mass 0.001; visual box size=0.001 0.001 0.001
- link FL_calf: mass 0.12532 -> 0.23; geometry collision box size=0.02 0.02 0.08; collision box size=0.02 0.02 0.18
- link FL_hip: mass 0.56406 -> 1.6; geometry visual mesh filename=package://mz_description/meshes/FL_hip.dae scale=1 1 1
- link FL_thigh: mass 0.72376 -> 2.7; geometry collision box size=0.04 0.025 0.30; visual mesh filename=package://mz_description/meshes/thigh_mirror.dae scale=1 1 1
- link FR_calf: mass 0.12532 -> 0.23; geometry collision box size=0.02 0.02 0.08; collision box size=0.02 0.02 0.18
- link FR_hip: mass 0.56406 -> 1.6; geometry visual mesh filename=package://mz_description/meshes/FR_hip.dae scale=1 1 1
- link FR_thigh: mass 0.72376 -> 2.7; geometry collision box size=0.04 0.025 0.30; visual mesh filename=package://mz_description/meshes/thigh.dae scale=1 1 1
- link RL_calf: mass 0.12532 -> 0.23; geometry collision box size=0.02 0.02 0.08; collision box size=0.02 0.02 0.18
- link RL_hip: mass 0 -> 1.6; geometry visual mesh filename=package://mz_description/meshes/RL_hip.dae scale=1 1 1
- link RL_thigh: mass 0.72376 -> 2.7; geometry collision box size=0.04 0.025 0.30; visual mesh filename=package://mz_description/meshes/thigh_mirror.dae scale=1 1 1
- link RR_calf: mass 0.12532 -> 0.23; geometry collision box size=0.02 0.02 0.08; collision box size=0.02 0.02 0.18
- link RR_hip: mass 0.56406 -> 1.6; geometry visual mesh filename=package://mz_description/meshes/RR_hip.dae scale=1 1 1
- link RR_thigh: mass 0.72376 -> 2.7; geometry collision box size=0.04 0.025 0.30; visual mesh filename=package://mz_description/meshes/thigh.dae scale=1 1 1
- link trunk: mass 4.9532 -> 16.6; geometry collision box size=0.470 0.3 0.150; visual mesh filename=package://mz_description/meshes/trunk.dae scale=1 1 1
Joints:
- added joint FL_hip_fixed: type fixed, parent FL_hip, child FL_thigh_shoulder, origin xyz=0 0.081 0 rpy=0 0 0
- added joint FR_hip_fixed: type fixed, parent FR_hip, child FR_thigh_shoulder, origin xyz=0 -0.081 0 rpy=0 0 0
- added joint RL_hip_fixed: type fixed, parent RL_hip, child RL_thigh_shoulder, origin xyz=0 0.081 0 rpy=0 0 0
- added joint RR_hip_fixed: type fixed, parent RR_hip, child RR_thigh_shoulder, origin xyz=0 -0.081 0 rpy=0 0 0
- added joint imu_joint: type fixed, parent trunk, child imu_link, origin xyz=0 0 0 rpy=0 0 0
- joint FL_calf_joint: axis 0 -1 0 -> 0 1 0; limit lower=-3.14 upper=3.14 effort=20 velocity=50 -> lower=-2.8099 upper=-1.0297 effort=60 velocity=9
- joint FL_foot_fixed: child FL_FOOT -> FL_foot
- joint FL_hip_joint: axis -1 0 0 -> 1 0 0; limit lower=-3.14 upper=3.14 effort=20 velocity=50 -> lower=-1.04 upper=1.04 effort=60 velocity=9
- joint FL_thigh_joint: axis 0 -1 0 -> 0 1 0; limit lower=-3.14 upper=3.14 effort=20 velocity=50 -> lower=-1.482 upper=3.9269 effort=60 velocity=9
- joint FR_calf_joint: axis 0 -1 0 -> 0 1 0; limit lower=-3.14 upper=3.14 effort=20 velocity=50 -> lower=-2.8099 upper=-1.0297 effort=60 velocity=9
- joint FR_foot_fixed: child FR_FOOT -> FR_foot; origin xyz=0 0 -0.305 rpy=0 0 0 -> xyz=0 0 -0.302 rpy=0 0 0
- joint FR_hip_joint: axis -1 0 0 -> 1 0 0; limit lower=-3.14 upper=3.14 effort=20 velocity=50 -> lower=-1.04 upper=1.04 effort=60 velocity=9
- joint FR_thigh_joint: limit lower=-3.14 upper=3.14 effort=20 velocity=50 -> lower=-1.482 upper=3.9269 effort=60 velocity=9
- joint RL_calf_joint: axis 0 -1 0 -> 0 1 0; limit lower=-3.14 upper=3.14 effort=20 velocity=50 -> lower=-2.8099 upper=-1.0297 effort=60 velocity=9
- joint RL_foot_fixed: child RL_FOOT -> RL_foot
- joint RL_hip_joint: limit lower=-3.14 upper=3.14 effort=20 velocity=50 -> lower=-1.04 upper=1.04 effort=60 velocity=9
- joint RL_thigh_joint: axis 0 -1 0 -> 0 1 0; limit lower=-3.14 upper=3.14 effort=20 velocity=50 -> lower=-0.6981 upper=4.7123 effort=60 velocity=9
- joint RR_calf_joint: axis 0 -1 0 -> 0 1 0; limit lower=-3.14 upper=3.14 effort=20 velocity=50 -> lower=-2.8099 upper=-1.0297 effort=60 velocity=9
- joint RR_foot_fixed: child RR_FOOT -> RR_foot
- joint RR_hip_joint: limit lower=-3.14 upper=3.14 effort=20 velocity=50 -> lower=-1.04 upper=1.04 effort=60 velocity=9
- joint RR_thigh_joint: limit lower=-3.14 upper=3.14 effort=20 velocity=50 -> lower=-0.6981 upper=4.7123 effort=60 velocity=9
