Commit message: fix trunk mass com

File: src/robots/b2_description/xacro/robot.xacro (robot description, xacro)
@@ -45,5 +45,5 @@
         </collision>
         <inertial>
-        <origin rpy="0 0 0" xyz="0.038238 -0.0086038 -0.0003117"/>
+        <origin rpy="0 0 0" xyz="0.1 -0.05 -0.0003117"/>
         <mass value="16.6"/>
         <inertia ixx="0.124986" ixy="-2.879308e-04" ixz="0.001458170" iyy="0.491519" iyz="-6.43446e-04" izz="0.5473926"/>

Commit message: 删除calf关节多个碰撞体积,提高real_time_rate

File: src/robots/b2_description/xacro/robot.xacro (robot description, xacro)
@@ -131,15 +131,15 @@
         </visual>
         <collision>
-        <origin xyz="0.018 0 -0.11" rpy="0 -0.30 0" />
-        <geometry>
-            <box size= "0.02 0.02 0.18"/>
-        </geometry>
-        </collision>
-        <collision>
+        <origin xyz="0.018 0 -0.16" rpy="0 -0.10 0" />
+        <geometry>
+            <box size= "0.02 0.02 0.24"/>
+        </geometry>
+        </collision>
+        <!-- <collision>
         <origin xyz="0.03 0 -0.245" rpy="0 0.35 0" />
         <geometry>
-            <box size= "0.02 0.02 0.08"/>
-        </geometry>
-        </collision>
+            "<box size= "0.02 0.02 0.06"/>
+        </geometry>
+        </collision> -->
         <inertial>
         <origin rpy="0 0 0" xyz="0.0079835 -6.7794E-06 -0.18022"/>
@@ -255,15 +255,15 @@
         </visual>
         <collision>
-        <origin xyz="0.018 0 -0.11" rpy="0 -0.30 0" />
-        <geometry>
-            <box size= "0.02 0.02 0.18"/>
-        </geometry>
-        </collision>
-        <collision>
+        <origin xyz="0.018 0 -0.16" rpy="0 -0.10 0" />
+        <geometry>
+            <box size= "0.02 0.02 0.24"/>
+        </geometry>
+        </collision>
+        <!-- <collision>
         <origin xyz="0.03 0 -0.245" rpy="0 0.35 0" />
         <geometry>
-            <box size= "0.02 0.02 0.08"/>
-        </geometry>
-        </collision>
+            "<box size= "0.02 0.02 0.06"/>
+        </geometry>
+        </collision> -->
         <inertial>
         <origin rpy="0 0 0" xyz="0.0079835 -6.7598E-06 -0.18022"/>
@@ -378,15 +378,15 @@
         </visual>
         <collision>
-        <origin xyz="0.018 0 -0.11" rpy="0 -0.30 0" />
-        <geometry>
-            <box size= "0.02 0.02 0.18"/>
-        </geometry>
-        </collision>
-        <collision>
+        <origin xyz="0.018 0 -0.16" rpy="0 -0.10 0" />
+        <geometry>
+            <box size= "0.02 0.02 0.24"/>
+        </geometry>
+        </collision>
+        <!-- <collision>
         <origin xyz="0.03 0 -0.245" rpy="0 0.35 0" />
         <geometry>
-            <box size= "0.02 0.02 0.08"/>
-        </geometry>
-        </collision>
+            "<box size= "0.02 0.02 0.06"/>
+        </geometry>
+        </collision> -->
         <inertial>
         <origin rpy="0 0 0" xyz="0.0079835 -6.7795E-06 -0.18022"/>
@@ -502,15 +502,15 @@
         </visual>
         <collision>
-        <origin xyz="0.018 0 -0.11" rpy="0 -0.30 0" />
-        <geometry>
-            <box size= "0.02 0.02 0.18"/>
-        </geometry>
-        </collision>
-        <collision>
+        <origin xyz="0.018 0 -0.16" rpy="0 -0.10 0" />
+        <geometry>
+            <box size= "0.02 0.02 0.24"/>
+        </geometry>
+        </collision>
+        <!-- <collision>
         <origin xyz="0.03 0 -0.245" rpy="0 0.35 0" />
         <geometry>
-            <box size= "0.02 0.02 0.08"/>
-        </geometry>
-        </collision>
+            "<box size= "0.02 0.02 0.06"/>
+        </geometry>
+        </collision> -->
         <inertial>
         <origin rpy="0 0 0" xyz="0.0079835 -6.7801E-06 -0.18022"/>

Commit message: 根据实物减小质心偏移程度

File: src/robots/b2_description/xacro/robot.xacro (robot description, xacro)
@@ -45,5 +45,5 @@
         </collision>
         <inertial>
-        <origin rpy="0 0 0" xyz="0.1 -0.05 -0.0003117"/>
+        <origin rpy="0 0 0" xyz="0.05 -0.025 -0.0003117"/>
         <mass value="16.6"/>
         <inertia ixx="0.124986" ixy="-2.879308e-04" ixz="0.001458170" iyy="0.491519" iyz="-6.43446e-04" izz="0.5473926"/>

Commit message: 修正重心位置

File: src/robots/b2_description/xacro/robot.xacro (robot description, xacro)
@@ -45,5 +45,5 @@
         </collision>
         <inertial>
-        <origin rpy="0 0 0" xyz="0.05 -0.025 -0.0003117"/>
+        <origin rpy="0 0 0" xyz="0.04 -0.02 -0.0003117"/>
         <mass value="16.6"/>
         <inertia ixx="0.124986" ixy="-2.879308e-04" ixz="0.001458170" iyy="0.491519" iyz="-6.43446e-04" izz="0.5473926"/>
