Commit message: 将中型四足的xacro文件重新校准

File: src/robots/mz_description/xacro/robot.xacro (robot description, xacro)
@@ -2,5 +2,5 @@
 <robot name="mz_description" xmlns:xacro="http://www.ros.org/wiki/xacro">
     <xacro:include filename="$(find mz_description)/xacro/const.xacro"/>
-    <xacro:include filename="$(find mz_description)/xacro/materials.xacro"/>
+    <!-- <xacro:include filename="$(find mz_description)/xacro/materials.xacro"/> -->
     <xacro:include filename="$(find mz_description)/xacro/leg.xacro"/>
     <xacro:include filename="$(find mz_description)/xacro/gazebo.xacro"/>
@@ -8,4 +8,16 @@
     <!-- Rotor related joint and link is only for demonstrate location. -->
     <!-- Actually, the rotor will rotate and the joint is not fixed. Reduction ratio should be considered. -->
+    <material name="blue">
+        <color rgba="0.0 0.0 0.8 1.0"/>
+    </material>
+    <material name="green">
+        <color rgba="0.0 0.8 0.0 1.0"/>
+    </material>
+    <material name="silver">
+        <color rgba="0.913725490196 0.913725490196 0.847058823529 0.5"/>
+    </material>
+    <material name="red">
+        <color rgba="0.8 0.0 0.0 1.0"/>
+    </material>
     <!-- Debug mode will hung up the robot, use "true" or "false" to switch it. -->
     <xacro:if value="$(arg DEBUG)">
@@ -39,4 +51,5 @@
         </visual>
         <collision>
+        <!-- trunk mesh com mark offset is 0.075 -->
         <origin rpy="0 0 0" xyz="0 0 0.075"/>
         <geometry>
@@ -45,16 +58,37 @@
         </collision>
         <inertial>
-        <origin rpy="0 0 0" xyz="0.04 -0.02 -0.0003117"/>
-        <mass value="16.6"/>
-        <inertia ixx="0.124986" ixy="-2.879308e-04" ixz="0.001458170" iyy="0.491519" iyz="-6.43446e-04" izz="0.5473926"/>
-        </inertial>
-    </link>
+        <origin rpy="0 0 0" xyz="0.0 0.0 0.0"/>
+        <mass value="16.28"/>
+        <inertia ixx="0.116459" ixy="0" ixz="0" iyy="0.519331" iyz="0" izz="0.583368"/>
+        </inertial>
+    </link>
+    <joint name="imu_joint" type="fixed">
+        <parent link="trunk"/>
+        <child link="imu_link"/>
+        <origin rpy="0 0 0" xyz="0 0 0"/>
+    </joint>
+    <link name="imu_link">
+        <inertial>
+        <mass value="0.001"/>
+        <origin rpy="0 0 0" xyz="0 0 0"/>
+        <inertia ixx="0.000001" ixy="0" ixz="0" iyy="0.000001" iyz="0" izz="0.000001"/>
+        </inertial>
+        <visual>
+        <origin rpy="0 0 0" xyz="0 0 0"/>
+        <geometry>
+            <box size="0.001 0.001 0.001"/>
+        </geometry>
+        <material name="silver"/>
+        </visual>
+    </link>
+    <!-- FR Leg -->
     <joint name="FR_hip_joint" type="revolute">
-        <origin rpy="0 0 0" xyz="0.22626 -0.070008 0.075"/>
+        <!-- trunk com offset is 0.075 -->
+        <origin rpy="0 0 0" xyz="0.22624 -0.07 0.075"/>
         <parent link="trunk"/>
         <child link="FR_hip"/>
         <axis xyz="1 0 0"/>
         <dynamics damping="0" friction="0"/>
-        <limit effort="60" lower="-1.04" upper="1.04" velocity="9"/>
+        <limit effort="67" lower="-1.04" upper="1.04" velocity="15"/>
     </joint>
     <link name="FR_hip">
@@ -67,22 +101,8 @@
         </visual>
         <inertial>
-        <origin rpy="0 0 0" xyz="0.083541 -0.0016537 1.2994E-05"/>
+        <origin rpy="0 0 0" xyz="0.08 -0.00177 0.00001"/>
         <mass value="1.6"/>
-        <inertia ixx="0.001582101" ixy="-0.0001151304" ixz="-4.046387E-06" iyy="0.002797035" iyz="0.000004285818" izz="0.001731282"/>
-        </inertial>
-    </link>
-    <joint name="FR_hip_fixed" type="fixed">
-        <origin rpy="0 0 0" xyz="0 -0.081 0"/>
-        <parent link="FR_hip"/>
-        <child link="FR_thigh_shoulder"/>
-    </joint>
-    <!-- this link is only for collision -->
-    <link name="FR_thigh_shoulder">
-        <!-- <collision>
-        <origin rpy="1.57079632679 0 0" xyz="0 0 0"/>
-        <geometry>
-            <cylinder length="0.032" radius="0.041"/>
-        </geometry>
-        </collision> -->
+        <inertia ixx="0.00173144" ixy="0" ixz="0" iyy="0.01332646" iyz="0" izz="0.01241473"/>
+        </inertial>
     </link>
     <joint name="FR_thigh_joint" type="revolute">
@@ -92,5 +112,5 @@
         <axis xyz="0 1 0"/>
         <dynamics damping="0" friction="0"/>
-        <limit effort="60" lower="-1.482" upper="3.9269" velocity="9"/>
+        <limit effort="67" lower="-1.482" upper="3.9269" velocity="15"/>
     </joint>
     <link name="FR_thigh">
@@ -109,7 +129,7 @@
         </collision>
         <inertial>
-        <origin rpy="0 0 0" xyz="-0.0027386 -0.061044 -0.025431"/>
+        <origin rpy="0 0 0" xyz="-0.00401 -0.06043 -0.03327"/>
         <mass value="2.7"/>
-        <inertia ixx="0.0370827" ixy="-0.0005225046" ixz="-0.002171109" iyy="0.03654717" iyz="-0.004972422" izz="0.004880799"/>
+        <inertia ixx="0.03077371" ixy="0" ixz="0" iyy="0.022321" iyz="0" izz="0.012608"/>
         </inertial>
     </link>
@@ -120,5 +140,5 @@
         <axis xyz="0 1 0"/>
         <dynamics damping="0" friction="0"/>
-        <limit effort="60" lower="-2.8099" upper="-1.0297" velocity="9"/>
+        <limit effort="67" lower="-2.8099" upper="-1.0297" velocity="15"/>
     </joint>
     <link name="FR_calf">
@@ -136,18 +156,12 @@
         </geometry>
         </collision>
-        <!-- <collision>
-        <origin xyz="0.03 0 -0.245" rpy="0 0.35 0" />
-        <geometry>
-            "<box size= "0.02 0.02 0.06"/>
-        </geometry>
-        </collision> -->
-        <inertial>
-        <origin rpy="0 0 0" xyz="0.0079835 -6.7794E-06 -0.18022"/>
+        <inertial>
+        <origin rpy="0 0 0" xyz="0.01038 0 -0.072"/>
         <mass value="0.23"/>
-        <inertia ixx="0.00650717" ixy="0.0" ixz="0.0003660643" iyy="0.006566385" iyz="0.0" izz="0.0001884405"/>
+        <inertia ixx="0.012939" ixy="0" ixz="0" iyy="0.012861" iyz="0" izz="0.000437"/>
         </inertial>
     </link>
     <joint name="FR_foot_fixed" type="fixed" dont_collapse="true">
-        <origin rpy="0 0 0" xyz="0 0 -0.302"/>
+        <origin rpy="0 0 0" xyz="0 0 -0.3"/>
         <parent link="FR_calf"/>
         <child link="FR_foot"/>
@@ -164,25 +178,27 @@
         <origin rpy="0 0 0" xyz="0 0 0"/>
         <geometry>
-            <!-- <sphere radius="0.02"/> -->
             <sphere radius="0.0235"/>
         </geometry>
         </collision>
         <inertial>
+        <origin rpy="0 0 0" xyz="0 0 0"/>
         <mass value="0.07"/>
-        <inertia ixx="0.00002111109" ixy="0.0" ixz="0.000006111105" iyy="0.000022777755" iyz="0.0" izz="0.00002333331"/>
-        </inertial>
-    </link>
+        <inertia ixx="0.00002" ixy="0" ixz="0" iyy="0.00002" iyz="0" izz="0.00002"/>
+        </inertial>
+    </link>
+    <!-- FR Leg end -->
+    <!-- FL Leg -->
     <joint name="FL_hip_joint" type="revolute">
-        <origin rpy="0 0 0" xyz="0.22626 0.069992 0.075"/>
+        <!-- trunk com offset is 0.075 -->
+        <origin rpy="0 0 0" xyz="0.22624 0.07 0.075"/>
         <parent link="trunk"/>
         <child link="FL_hip"/>
         <axis xyz="1 0 0"/>
         <dynamics damping="0" friction="0"/>
-        <limit effort="60" lower="-1.04" upper="1.04" velocity="9"/>
+        <limit effort="67" lower="-1.04" upper="1.04" velocity="15"/>
     </joint>
     <link name="FL_hip">
         <visual>
-        <!-- the same as a1 -->
-        <origin rpy="0 0 0" xyz="0 0 0"/>
+        <origin xyz="0 0 0" rpy="0 0 0" />
         <geometry>
             <mesh filename="package://mz_description/meshes/FL_hip.dae" scale="1 1 1"/>
@@ -191,22 +207,8 @@
         </visual>
         <inertial>
-        <origin rpy="0 0 0" xyz="0.083541 0.0016537 -1.2994E-05"/>
+        <origin rpy="0 0 0" xyz="0.08 0.00177 0.00001"/>
         <mass value="1.6"/>
-        <inertia ixx="0.001986561" ixy="0.000042857612" ixz="-0.00000022566089" iyy="0.002917609" iyz="0.00000000239428" izz="0.002219916"/>
-        </inertial>
-    </link>
-    <joint name="FL_hip_fixed" type="fixed">
-        <origin rpy="0 0 0" xyz="0 0.081 0"/>
-        <parent link="FL_hip"/>
-        <child link="FL_thigh_shoulder"/>
-    </joint>
-    <!-- this link is only for collision -->
-    <link name="FL_thigh_shoulder">
-        <!-- <collision>
-        <origin rpy="1.57079632679 0 0" xyz="0 0 0"/>
-        <geometry>
-            <cylinder length="0.032" radius="0.041"/>
-        </geometry>
-        </collision> -->
+        <inertia ixx="0.00173144" ixy="0" ixz="0" iyy="0.01332646" iyz="0" izz="0.01241473"/>
+        </inertial>
     </link>
     <joint name="FL_thigh_joint" type="revolute">
@@ -216,5 +218,5 @@
         <axis xyz="0 1 0"/>
         <dynamics damping="0" friction="0"/>
-        <limit effort="60" lower="-1.482" upper="3.9269" velocity="9"/>
+        <limit effort="67" lower="-1.482" upper="3.9269" velocity="15"/>
     </joint>
     <link name="FL_thigh">
@@ -233,7 +235,7 @@
         </collision>
         <inertial>
-        <origin rpy="0 0 0" xyz="-0.0027198 0.061044 -0.025411"/>
+        <origin rpy="0 0 0" xyz="-0.00401 0.06043 -0.03327"/>
         <mass value="2.7"/>
-        <inertia ixx="0.0370822" ixy="0.0005224988" ixz="-0.002171101" iyy="0.03654652" iyz="0.00497237" izz="0.004880707"/>
+        <inertia ixx="0.03077371" ixy="0" ixz="0" iyy="0.022321" iyz="0" izz="0.012608"/>
         </inertial>
     </link>
@@ -244,5 +246,5 @@
         <axis xyz="0 1 0"/>
         <dynamics damping="0" friction="0"/>
-        <limit effort="60" lower="-2.8099" upper="-1.0297" velocity="9"/>
+        <limit effort="67" lower="-2.8099" upper="-1.0297" velocity="15"/>
     </joint>
     <link name="FL_calf">
@@ -260,18 +262,12 @@
         </geometry>
         </collision>
-        <!-- <collision>
-        <origin xyz="0.03 0 -0.245" rpy="0 0.35 0" />
-        <geometry>
-            "<box size= "0.02 0.02 0.06"/>
-        </geometry>
-        </collision> -->
-        <inertial>
-        <origin rpy="0 0 0" xyz="0.0079835 -6.7598E-06 -0.18022"/>
+        <inertial>
+        <origin rpy="0 0 0" xyz="0.01038 0 -0.072"/>
         <mass value="0.23"/>
-        <inertia ixx="0.006507178" ixy="0.0" ixz="0.0003660643" iyy="0.006566385" iyz="0.0" izz="0.0001884405"/>
+        <inertia ixx="0.012939" ixy="0" ixz="0" iyy="0.012861" iyz="0" izz="0.000437"/>
         </inertial>
     </link>
     <joint name="FL_foot_fixed" type="fixed" dont_collapse="true">
-        <origin rpy="0 0 0" xyz="0 0 -0.302"/>
+        <origin rpy="0 0 0" xyz="0 0 -0.3"/>
         <parent link="FL_calf"/>
         <child link="FL_foot"/>
@@ -281,5 +277,5 @@
         <origin rpy="0 0 0" xyz="0 0 0"/>
         <geometry>
-            <sphere radius="0.015"/>
+            <sphere radius="0.01"/>
         </geometry>
         <material name="silver"/>
@@ -292,20 +288,23 @@
         </collision>
         <inertial>
+        <origin rpy="0 0 0" xyz="0 0 0"/>
         <mass value="0.07"/>
-        <!-- the same as a1 -->
-        <inertia ixx="2.1111e-05" ixy="0.0" ixz="0.000006111105" iyy="0.000022777755" iyz="0.0" izz="0.00002333331"/>
-        </inertial>
-    </link>
+        <inertia ixx="0.00002" ixy="0" ixz="0" iyy="0.00002" iyz="0" izz="0.00002"/>
+        </inertial>
+    </link>
+    <!-- FL Leg end -->
+    <!-- RR Leg -->
     <joint name="RR_hip_joint" type="revolute">
-        <origin rpy="0 0 0" xyz="-0.22624 -0.070008 0.075"/>
+        <!-- trunk com offset is 0.075 -->
+        <origin rpy="0 0 0" xyz="-0.22624 -0.07 0.075"/>
         <parent link="trunk"/>
         <child link="RR_hip"/>
         <axis xyz="1 0 0"/>
         <dynamics damping="0" friction="0"/>
-        <limit effort="60" lower="-1.04" upper="1.04" velocity="9"/>
+        <limit effort="67" lower="-1.04" upper="1.04" velocity="15"/>
     </joint>
     <link name="RR_hip">
         <visual>
-        <origin rpy="0 0 0" xyz="0 0 0"/>
+        <origin xyz="0 0 0" rpy="0 0 0" />
         <geometry>
             <mesh filename="package://mz_description/meshes/RR_hip.dae" scale="1 1 1"/>
@@ -314,22 +313,8 @@
         </visual>
         <inertial>
-        <origin rpy="0 0 0" xyz="-0.083541 -0.0016537 -1.2994E-05"/>
+        <origin rpy="0 0 0" xyz="-0.08 -0.00177 0.00001"/>
         <mass value="1.6"/>
-        <inertia ixx="0.001986561" ixy="0.00004285820" ixz="0.0000002256640" iyy="0.002917650" iyz="-0.000000002394313" izz="0.002219947"/>
-        </inertial>
-    </link>
-    <joint name="RR_hip_fixed" type="fixed">
-        <origin rpy="0 0 0" xyz="0 -0.081 0"/>
-        <parent link="RR_hip"/>
-        <child link="RR_thigh_shoulder"/>
-    </joint>
-    <!-- this link is only for collision -->
-    <link name="RR_thigh_shoulder">
-        <!-- <collision>
-        <origin rpy="1.57079632679 0 0" xyz="0 0 0"/>
-        <geometry>
-            <cylinder length="0.032" radius="0.041"/>
-        </geometry>
-        </collision> -->
+        <inertia ixx="0.00173144" ixy="0" ixz="0" iyy="0.01332646" iyz="0" izz="0.01241473"/>
+        </inertial>
     </link>
     <joint name="RR_thigh_joint" type="revolute">
@@ -339,5 +324,5 @@
         <axis xyz="0 1 0"/>
         <dynamics damping="0" friction="0"/>
-        <limit effort="60" lower="-0.6981" upper="4.7123" velocity="9"/>
+        <limit effort="67" lower="-1.482" upper="3.9269" velocity="15"/>
     </joint>
     <link name="RR_thigh">
@@ -356,7 +341,7 @@
         </collision>
         <inertial>
-        <origin rpy="0 0 0" xyz="-0.0027386 -0.061044 -0.025431"/>
+        <origin rpy="0 0 0" xyz="-0.00401 -0.06043 -0.03327"/>
         <mass value="2.7"/>
-        <inertia ixx="0.0370827" ixy="-0.000522505" ixz="-0.002171130" iyy="0.03654701" iyz="-0.00497243" izz="0.00488077"/>
+        <inertia ixx="0.03077371" ixy="0" ixz="0" iyy="0.022321" iyz="0" izz="0.012608"/>
         </inertial>
     </link>
@@ -367,5 +352,5 @@
         <axis xyz="0 1 0"/>
         <dynamics damping="0" friction="0"/>
-        <limit effort="60" lower="-2.8099" upper="-1.0297" velocity="9"/>
+        <limit effort="67" lower="-2.8099" upper="-1.0297" velocity="15"/>
     </joint>
     <link name="RR_calf">
@@ -383,19 +368,12 @@
         </geometry>
         </collision>
-        <!-- <collision>
-        <origin xyz="0.03 0 -0.245" rpy="0 0.35 0" />
-        <geometry>
-            "<box size= "0.02 0.02 0.06"/>
-        </geometry>
-        </collision> -->
-        <inertial>
-        <origin rpy="0 0 0" xyz="0.0079835 -6.7795E-06 -0.18022"/>
+        <inertial>
+        <origin rpy="0 0 0" xyz="0.01038 0 -0.072"/>
         <mass value="0.23"/>
-        <inertia ixx="0.00650709" ixy="0.0" ixz="0.0003660599" iyy="0.006566306" iyz="0.0" izz="0.0001884383"/>
-        <!-- <inertia ixx="0.0034783165033113" ixy="0.0" ixz="-2.095735099337748e-4" iyy="0.0035020471523179" iyz="0.0" izz="4.622113907284768e-5" /> -->
+        <inertia ixx="0.012939" ixy="0" ixz="0" iyy="0.012861" iyz="0" izz="0.000437"/>
         </inertial>
     </link>
     <joint name="RR_foot_fixed" type="fixed" dont_collapse="true">
-        <origin rpy="0 0 0" xyz="0 0 -0.302"/>
+        <origin rpy="0 0 0" xyz="0 0 -0.3"/>
         <parent link="RR_calf"/>
         <child link="RR_foot"/>
@@ -416,16 +394,19 @@
         </collision>
         <inertial>
+        <origin rpy="0 0 0" xyz="0 0 0"/>
         <mass value="0.07"/>
-        <!-- the same as a1 -->
-        <inertia ixx="2.11111e-05" ixy="0.0" ixz="0.000006111105" iyy="0.00002277775" iyz="0.0" izz="0.00002333331"/>
-        </inertial>
-    </link>
+        <inertia ixx="0.00002" ixy="0" ixz="0" iyy="0.00002" iyz="0" izz="0.00002"/>
+        </inertial>
+    </link>
+    <!-- RR Leg end -->
+    <!-- RL Leg -->
     <joint name="RL_hip_joint" type="revolute">
-        <origin rpy="0 0 0" xyz="-0.22624 0.069992 0.075"/>
+        <!-- trunk com offset is 0.075 -->
+        <origin rpy="0 0 0" xyz="-0.22624 0.07 0.075"/>
         <parent link="trunk"/>
         <child link="RL_hip"/>
         <axis xyz="1 0 0"/>
         <dynamics damping="0" friction="0"/>
-        <limit effort="60" lower="-1.04" upper="1.04" velocity="9"/>
+        <limit effort="67" lower="-1.04" upper="1.04" velocity="15"/>
     </joint>
     <link name="RL_hip">
@@ -438,22 +419,8 @@
         </visual>
         <inertial>
-        <origin rpy="0 0 0" xyz="0.0037743 0.0038894 7.8535E-05"/>
+        <origin rpy="0 0 0" xyz="-0.08 0.00177 0.00001"/>
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
Commit message: 以Gazebo可视化界面为评估参考，根据实物重新校准中型mz的urdf模型文件。经过训练、仿真、实物测试，该urdf文件相比之前的各版本都更贴近实物。

File: src/robots/mz_description/xacro/robot.xacro (robot description, xacro)
@@ -58,7 +58,7 @@
         </collision>
         <inertial>
-        <origin rpy="0 0 0" xyz="0.0 0.0 0.0"/>
+        <origin rpy="0 0 0" xyz="0.0 0.0 0.075"/>
         <mass value="16.28"/>
-        <inertia ixx="0.116459" ixy="0" ixz="0" iyy="0.519331" iyz="0" izz="0.583368"/>
+        <inertia ixx="0.1487" ixy="0" ixz="0" iyy="0.3264" iyz="0" izz="0.4219"/>
         </inertial>
     </link>
@@ -130,5 +130,5 @@
             <origin rpy="0 0 0" xyz="-0.0027386 -0.061044 -0.025431"/>
             <mass value="2.7"/>
-            <inertia ixx="0.0370827" ixy="-0.0005225046" ixz="-0.002171109" iyy="0.03654717" iyz="-0.004972422" izz="0.004880799"/>
+            <inertia ixx="0.03473" ixy="0.0" ixz="0.0" iyy="0.03473" iyz="0.0" izz="0.003689"/>
         </inertial>
     </link>
@@ -158,5 +158,5 @@
             <origin rpy="0 0 0" xyz="0.0079835 -6.7794E-06 -0.18022"/>
             <mass value="0.23"/>
-            <inertia ixx="0.00650717" ixy="0.0" ixz="0.0003660643" iyy="0.006566385" iyz="0.0" izz="0.0001884405"/>
+            <inertia ixx="0.002770" ixy="0" ixz="0" iyy="0.002764" iyz="0" izz="0.000041"/>
         </inertial>
     </link>
@@ -177,5 +177,5 @@
         <origin rpy="0 0 0" xyz="0 0 0"/>
         <geometry>
-            <sphere radius="0.0235"/>
+            <sphere radius="0.025"/>
         </geometry>
         </collision>
@@ -236,5 +236,5 @@
             <origin rpy="0 0 0" xyz="-0.0027198 0.061044 -0.025411"/>
             <mass value="2.7"/>
-            <inertia ixx="0.0370822" ixy="0.0005224988" ixz="-0.002171101" iyy="0.03654652" iyz="0.00497237" izz="0.004880707"/>
+            <inertia ixx="0.03473" ixy="0.0" ixz="0.0" iyy="0.03473" iyz="0.0" izz="0.003689"/>
         </inertial>
     </link>
@@ -264,5 +264,5 @@
             <origin rpy="0 0 0" xyz="0.0079835 -6.7598E-06 -0.18022"/>
             <mass value="0.23"/>
-            <inertia ixx="0.006507178" ixy="0.0" ixz="0.0003660643" iyy="0.006566385" iyz="0.0" izz="0.0001884405"/>
+            <inertia ixx="0.002770" ixy="0" ixz="0" iyy="0.002764" iyz="0" izz="0.000041"/>
         </inertial>
     </link>
@@ -283,5 +283,5 @@
         <origin rpy="0 0 0" xyz="0 0 0"/>
         <geometry>
-            <sphere radius="0.0235"/>
+            <sphere radius="0.025"/>
         </geometry>
         </collision>
@@ -341,5 +341,5 @@
             <origin rpy="0 0 0" xyz="-0.0027386 -0.061044 -0.025431"/>
             <mass value="2.7"/>
-            <inertia ixx="0.0370827" ixy="-0.000522505" ixz="-0.002171130" iyy="0.03654701" iyz="-0.00497243" izz="0.00488077"/>
+            <inertia ixx="0.03473" ixy="0.0" ixz="0.0" iyy="0.03473" iyz="0.0" izz="0.003689"/>
         </inertial>
     </link>
@@ -369,5 +369,5 @@
             <origin rpy="0 0 0" xyz="0.0079835 -6.7795E-06 -0.18022"/>
             <mass value="0.23"/>
-            <inertia ixx="0.00650709" ixy="0.0" ixz="0.0003660599" iyy="0.006566306" iyz="0.0" izz="0.0001884383"/>
+            <inertia ixx="0.002770" ixy="0" ixz="0" iyy="0.002764" iyz="0" izz="0.000041"/>
         </inertial>
     </link>
@@ -388,5 +388,5 @@
         <origin rpy="0 0 0" xyz="0 0 0"/>
         <geometry>
-            <sphere radius="0.0235"/>
+            <sphere radius="0.025"/>
         </geometry>
         </collision>
@@ -443,8 +443,8 @@
             </geometry>
         </collision>
-            <inertial>
+        <inertial>
             <origin rpy="0 0 0" xyz="-0.0027198 0.061044 -0.025411"/>
             <mass value="2.7"/>
-            <inertia ixx="0.0370827" ixy="0.000522504" ixz="-0.002171109" iyy="0.0365471" iyz="0.00497242" izz="0.004880799"/>
+            <inertia ixx="0.03473" ixy="0.0" ixz="0.0" iyy="0.03473" iyz="0.0" izz="0.003689"/>
         </inertial>
     </link>
@@ -474,5 +474,5 @@
             <origin rpy="0 0 0" xyz="0.0079835 -6.7801E-06 -0.18022"/>
             <mass value="0.23"/>
-            <inertia ixx="0.006507167" ixy="0.0" ixz="0.0003660637" iyy="0.006566375" iyz="0.0" izz="0.0001884402"/>
+            <inertia ixx="0.002770" ixy="0" ixz="0" iyy="0.002764" iyz="0" izz="0.000041"/>
         </inertial>
     </link>
@@ -493,5 +493,5 @@
         <origin rpy="0 0 0" xyz="0 0 0"/>
         <geometry>
-            <sphere radius="0.0235"/>
+            <sphere radius="0.025"/>
         </geometry>
         </collision>

Commit message: 将中型四足机器人urdf文件中hip关节的惯量积置零

File: src/robots/mz_description/xacro/robot.xacro (robot description, xacro)
@@ -102,5 +102,5 @@
             <origin rpy="0 0 0" xyz="0.083541 -0.0016537 -1.2994E-05"/>
             <mass value="1.6"/>
-            <inertia ixx="0.001986561" ixy="-0.000042857612" ixz="-0.00000022566" iyy="0.002917609" iyz="-0.00000000239428" izz="0.002219916"/>
+            <inertia ixx="0.001986561" ixy="0.0" ixz="0.0" iyy="0.002917609" iyz="0" izz="0.002219916"/>
         </inertial>
     </link>
@@ -208,5 +208,5 @@
             <origin rpy="0 0 0" xyz="0.083541 0.0016537 -1.2994E-05"/>
             <mass value="1.6"/>
-            <inertia ixx="0.001986561" ixy="0.000042857612" ixz="-0.00000022566089" iyy="0.002917609" iyz="0.00000000239428" izz="0.002219916"/>
+            <inertia ixx="0.001986561" ixy="0.0" ixz="0.0" iyy="0.002917609" iyz="0.0" izz="0.002219916"/>
         </inertial>
     </link>
@@ -313,5 +313,5 @@
             <origin rpy="0 0 0" xyz="-0.083541 -0.0016537 -1.2994E-05"/>
             <mass value="1.6"/>
-            <inertia ixx="0.001986561" ixy="0.00004285820" ixz="0.0000002256640" iyy="0.002917650" iyz="-0.000000002394313" izz="0.002219947"/>
+            <inertia ixx="0.001986561" ixy="0.0" ixz="0.0" iyy="0.002917650" iyz="0.0" izz="0.002219947"/>
         </inertial>
     </link>
@@ -418,5 +418,5 @@
             <origin rpy="0 0 0" xyz="-0.083541 0.0016537 -1.2994E-05"/>
             <mass value="1.6"/>
-            <inertia ixx="0.001986561" ixy="-0.00004285820" ixz="0.0000002256640" iyy="0.002917650" iyz="0.000000002394313" izz="0.002219916"/>
+            <inertia ixx="0.001986561" ixy="0.0" ixz="0.0" iyy="0.002917650" iyz="0.0" izz="0.002219916"/>
         </inertial>
     </link>
