Commit message: 按gazebo编辑器的转动惯量计算方法，更新了中型四足模型文件的转动惯量。

File: src/robots/mz_description/xacro/robot.xacro (robot description, xacro)
@@ -60,5 +60,5 @@
         <origin rpy="0 0 0" xyz="0.0 0.0 0.075"/>
         <mass value="16.28"/>
-        <inertia ixx="0.1487" ixy="0" ixz="0" iyy="0.3264" iyz="0" izz="0.4219"/>
+        <inertia ixx="0.115795" ixy="0" ixz="0" iyy="0.516939" iyz="0" izz="0.580354"/>
         </inertial>
     </link>
@@ -84,5 +84,6 @@
     <!-- FR Leg -->
     <joint name="FR_hip_joint" type="revolute">
-        <origin rpy="0 0 0" xyz="0.22626 -0.070008 0.075"/>
+        <!-- trunk com offset is 0.075 -->
+        <origin rpy="0 0 0" xyz="0.22624 -0.07 0.075"/>
         <parent link="trunk"/>
         <child link="FR_hip"/>
@@ -91,16 +92,17 @@
         <limit effort="67" lower="-1.04" upper="1.04" velocity="15"/>
     </joint>
+    <!-- 国庆节修改的hip关节模型 -->
     <link name="FR_hip">
         <visual>
-            <origin xyz="0 0 0" rpy="0 0 0" />
-            <geometry>
-                <mesh filename="package://mz_description/meshes/FR_hip.dae" scale="1 1 1"/>
-            </geometry>
-            <material name="silver"/>
-        </visual>
-        <inertial>
-            <origin rpy="0 0 0" xyz="0.083541 -0.0016537 -1.2994E-05"/>
-            <mass value="1.6"/>
-            <inertia ixx="0.001986561" ixy="0.0" ixz="0.0" iyy="0.002917609" iyz="0" izz="0.002219916"/>
+        <origin xyz="0 0 0" rpy="0 0 0" />
+        <geometry>
+            <mesh filename="package://mz_description/meshes/FR_hip.dae" scale="1 1 1"/>
+        </geometry>
+        <material name="silver"/>
+        </visual>
+        <inertial>
+        <origin rpy="0 0 0" xyz="0.08 -0.00177 0.00001"/>
+        <mass value="1.6"/>
+        <inertia ixx="0.001726" ixy="0" ixz="0" iyy="0.003117" iyz="0" izz="0.002200"/>
         </inertial>
     </link>
@@ -115,20 +117,20 @@
     <link name="FR_thigh">
         <visual>
-            <origin rpy="0 0 0" xyz="0 0 0"/>
-            <geometry>
-                <mesh filename="package://mz_description/meshes/thigh.dae" scale="1 1 1"/>
-            </geometry>
-            <material name="silver"/>
-        </visual>
-        <collision>
-            <origin xyz="-0.022 -0.094 -0.115" rpy="0 0 0" />
-            <geometry>
-                <box size="0.04 0.025 0.30"/>
-            </geometry>
-        </collision>
-        <inertial>
-            <origin rpy="0 0 0" xyz="-0.0027386 -0.061044 -0.025431"/>
-            <mass value="2.7"/>
-            <inertia ixx="0.03473" ixy="0.0" ixz="0.0" iyy="0.03473" iyz="0.0" izz="0.003689"/>
+        <origin rpy="0 0 0" xyz="0 0 0"/>
+        <geometry>
+            <mesh filename="package://mz_description/meshes/thigh.dae" scale="1 1 1"/>
+        </geometry>
+        <material name="silver"/>
+        </visual>
+        <collision>
+        <origin xyz="-0.022 -0.094 -0.115" rpy="0 0 0" />
+        <geometry>
+            <box size="0.04 0.025 0.30"/>
+        </geometry>
+        </collision>
+        <inertial>
+        <origin rpy="0 0 0" xyz="-0.00401 -0.06043 -0.03327"/>
+        <mass value="2.7"/>
+        <inertia ixx="0.019302" ixy="0" ixz="0" iyy="0.019614" iyz="0" izz="0.003767"/>
         </inertial>
     </link>
@@ -143,20 +145,20 @@
     <link name="FR_calf">
         <visual>
-            <origin rpy="0 0 0" xyz="0 0 0"/>
-            <geometry>
-                <mesh filename="package://mz_description/meshes/calf.dae" scale="1 1 1"/>
-            </geometry>
-            <material name="silver"/>
-        </visual>
-        <collision>
-            <origin xyz="0.018 0 -0.11" rpy="0 -0.30 0" />
-            <geometry>
-                <box size= "0.02 0.02 0.18"/>
-            </geometry>
-        </collision>
-        <inertial>
-            <origin rpy="0 0 0" xyz="0.0079835 -6.7794E-06 -0.18022"/>
-            <mass value="0.23"/>
-            <inertia ixx="0.002770" ixy="0" ixz="0" iyy="0.002764" iyz="0" izz="0.000041"/>
+        <origin rpy="0 0 0" xyz="0 0 0"/>
+        <geometry>
+            <mesh filename="package://mz_description/meshes/calf.dae" scale="1 1 1"/>
+        </geometry>
+        <material name="silver"/>
+        </visual>
+        <collision>
+        <origin xyz="0.018 0 -0.16" rpy="0 -0.10 0" />
+        <geometry>
+            <box size= "0.02 0.02 0.24"/>
+        </geometry>
+        </collision>
+        <inertial>
+        <origin rpy="0 0 0" xyz="0.01038 0 -0.072"/>
+        <mass value="0.23"/>
+        <inertia ixx="0.009492" ixy="0" ixz="0" iyy="0.009342" iyz="0" izz="0.000366"/>
         </inertial>
     </link>
@@ -177,5 +179,5 @@
         <origin rpy="0 0 0" xyz="0 0 0"/>
         <geometry>
-            <sphere radius="0.025"/>
+            <sphere radius="0.0235"/>
         </geometry>
         </collision>
@@ -189,5 +191,6 @@
     <!-- FL Leg -->
     <joint name="FL_hip_joint" type="revolute">
-        <origin rpy="0 0 0" xyz="0.22626 0.069992 0.075"/>
+        <!-- trunk com offset is 0.075 -->
+        <origin rpy="0 0 0" xyz="0.22624 0.07 0.075"/>
         <parent link="trunk"/>
         <child link="FL_hip"/>
@@ -196,17 +199,17 @@
         <limit effort="67" lower="-1.04" upper="1.04" velocity="15"/>
     </joint>
+    <!-- 国庆节修改的hip关节模型 -->
     <link name="FL_hip">
         <visual>
-        <!-- the same as a1 -->
-            <origin rpy="0 0 0" xyz="0 0 0"/>
-            <geometry>
-                <mesh filename="package://mz_description/meshes/FL_hip.dae" scale="1 1 1"/>
-            </geometry>
-            <material name="silver"/>
-        </visual>
-        <inertial>
-            <origin rpy="0 0 0" xyz="0.083541 0.0016537 -1.2994E-05"/>
-            <mass value="1.6"/>
-            <inertia ixx="0.001986561" ixy="0.0" ixz="0.0" iyy="0.002917609" iyz="0.0" izz="0.002219916"/>
+        <origin xyz="0 0 0" rpy="0 0 0" />
+        <geometry>
+            <mesh filename="package://mz_description/meshes/FL_hip.dae" scale="1 1 1"/>
+        </geometry>
+        <material name="silver"/>
+        </visual>
+        <inertial>
+        <origin rpy="0 0 0" xyz="0.08 0.00177 0.00001"/>
+        <mass value="1.6"/>
+        <inertia ixx="0.001726" ixy="0" ixz="0" iyy="0.003117" iyz="0" izz="0.002200"/>
         </inertial>
     </link>
@@ -221,20 +224,20 @@
     <link name="FL_thigh">
         <visual>
-            <origin rpy="0 0 0" xyz="0 0 0"/>
-            <geometry>
-                <mesh filename="package://mz_description/meshes/thigh_mirror.dae" scale="1 1 1"/>
-            </geometry>
-            <material name="silver"/>
-        </visual>
-        <collision>
-            <origin xyz="-0.022 0.094 -0.115" rpy="0 0 0" />
-            <geometry>
-                <box size="0.04 0.025 0.30"/>
-            </geometry>
-        </collision>
-        <inertial>
-            <origin rpy="0 0 0" xyz="-0.0027198 0.061044 -0.025411"/>
-            <mass value="2.7"/>
-            <inertia ixx="0.03473" ixy="0.0" ixz="0.0" iyy="0.03473" iyz="0.0" izz="0.003689"/>
+        <origin rpy="0 0 0" xyz="0 0 0"/>
+        <geometry>
+            <mesh filename="package://mz_description/meshes/thigh_mirror.dae" scale="1 1 1"/>
+        </geometry>
+        <material name="silver"/>
+        </visual>
+        <collision>
+        <origin xyz="-0.022 0.094 -0.115" rpy="0 0 0" />
+        <geometry>
+            <box size="0.04 0.025 0.30"/>
+        </geometry>
+        </collision>
+        <inertial>
+        <origin rpy="0 0 0" xyz="-0.00401 0.06043 -0.03327"/>
+        <mass value="2.7"/>
+        <inertia ixx="0.019302" ixy="0" ixz="0" iyy="0.019614" iyz="0" izz="0.003767"/>
         </inertial>
     </link>
@@ -249,20 +252,20 @@
     <link name="FL_calf">
         <visual>
-            <origin rpy="0 0 0" xyz="0 0 0"/>
-            <geometry>
-                <mesh filename="package://mz_description/meshes/calf.dae" scale="1 1 1"/>
-            </geometry>
-            <material name="silver"/>
-        </visual>
-        <collision>
-            <origin xyz="0.018 0 -0.11" rpy="0 -0.30 0" />
-            <geometry>
-                <box size= "0.02 0.02 0.18"/>
-            </geometry>
-        </collision>
-        <inertial>
-            <origin rpy="0 0 0" xyz="0.0079835 -6.7598E-06 -0.18022"/>
-            <mass value="0.23"/>
-            <inertia ixx="0.002770" ixy="0" ixz="0" iyy="0.002764" iyz="0" izz="0.000041"/>
+        <origin rpy="0 0 0" xyz="0 0 0"/>
+        <geometry>
+            <mesh filename="package://mz_description/meshes/calf.dae" scale="1 1 1"/>
+        </geometry>
+        <material name="silver"/>
+        </visual>
+        <collision>
+        <origin xyz="0.018 0 -0.16" rpy="0 -0.10 0" />
+        <geometry>
+            <box size= "0.02 0.02 0.24"/>
+        </geometry>
+        </collision>
+        <inertial>
+        <origin rpy="0 0 0" xyz="0.01038 0 -0.072"/>
+        <mass value="0.23"/>
+        <inertia ixx="0.009492" ixy="0" ixz="0" iyy="0.009342" iyz="0" izz="0.000366"/>
         </inertial>
     </link>
@@ -283,5 +286,5 @@
         <origin rpy="0 0 0" xyz="0 0 0"/>
         <geometry>
-            <sphere radius="0.025"/>
+            <sphere radius="0.0235"/>
         </geometry>
         </collision>
@@ -295,5 +298,6 @@
     <!-- RR Leg -->
     <joint name="RR_hip_joint" type="revolute">
-        <origin rpy="0 0 0" xyz="-0.22624 -0.070008 0.075"/>
+        <!-- trunk com offset is 0.075 -->
+        <origin rpy="0 0 0" xyz="-0.22624 -0.07 0.075"/>
         <parent link="trunk"/>
         <child link="RR_hip"/>
@@ -302,16 +306,17 @@
         <limit effort="67" lower="-1.04" upper="1.04" velocity="15"/>
     </joint>
+    <!-- 国庆节修改的hip关节模型 -->
     <link name="RR_hip">
         <visual>
-            <origin rpy="0 0 0" xyz="0 0 0"/>
-            <geometry>
-                <mesh filename="package://mz_description/meshes/RR_hip.dae" scale="1 1 1"/>
-            </geometry>
-            <material name="silver"/>
-        </visual>
-        <inertial>
-            <origin rpy="0 0 0" xyz="-0.083541 -0.0016537 -1.2994E-05"/>
-            <mass value="1.6"/>
-            <inertia ixx="0.001986561" ixy="0.0" ixz="0.0" iyy="0.002917650" iyz="0.0" izz="0.002219947"/>
+        <origin xyz="0 0 0" rpy="0 0 0" />
+        <geometry>
+            <mesh filename="package://mz_description/meshes/RR_hip.dae" scale="1 1 1"/>
+        </geometry>
+        <material name="silver"/>
+        </visual>
+        <inertial>
+        <origin rpy="0 0 0" xyz="-0.08 -0.00177 0.00001"/>
+        <mass value="1.6"/>
+        <inertia ixx="0.001726" ixy="0" ixz="0" iyy="0.003117" iyz="0" izz="0.002200"/>
         </inertial>
     </link>
@@ -322,24 +327,24 @@
         <axis xyz="0 1 0"/>
         <dynamics damping="0" friction="0"/>
-        <limit effort="67" lower="-0.6981" upper="4.7123" velocity="15"/>
+        <limit effort="67" lower="-1.482" upper="3.9269" velocity="15"/>
     </joint>
     <link name="RR_thigh">
         <visual>
-            <origin rpy="0 0 0" xyz="0 0 0"/>
-            <geometry>
-                <mesh filename="package://mz_description/meshes/thigh.dae" scale="1 1 1"/>
-            </geometry>
-            <material name="silver"/>
-        </visual>
-        <collision>
-            <origin xyz="-0.022 -0.094 -0.115" rpy="0 0 0" />
-            <geometry>
-                <box size="0.04 0.025 0.30"/>
-            </geometry>
-        </collision>
-        <inertial>
-            <origin rpy="0 0 0" xyz="-0.0027386 -0.061044 -0.025431"/>
-            <mass value="2.7"/>
-            <inertia ixx="0.03473" ixy="0.0" ixz="0.0" iyy="0.03473" iyz="0.0" izz="0.003689"/>
+        <origin rpy="0 0 0" xyz="0 0 0"/>
+        <geometry>
+            <mesh filename="package://mz_description/meshes/thigh.dae" scale="1 1 1"/>
+        </geometry>
+        <material name="silver"/>
+        </visual>
+        <collision>
+        <origin xyz="-0.022 -0.094 -0.115" rpy="0 0 0" />
+        <geometry>
+            <box size="0.04 0.025 0.30"/>
+        </geometry>
+        </collision>
+        <inertial>
+        <origin rpy="0 0 0" xyz="-0.00401 -0.06043 -0.03327"/>
+        <mass value="2.7"/>
+        <inertia ixx="0.019302" ixy="0" ixz="0" iyy="0.019614" iyz="0" izz="0.003767"/>
         </inertial>
     </link>
@@ -354,20 +359,20 @@
     <link name="RR_calf">
         <visual>
-            <origin rpy="0 0 0" xyz="0 0 0"/>
-            <geometry>
-                <mesh filename="package://mz_description/meshes/calf.dae" scale="1 1 1"/>
-            </geometry>
-            <material name="silver"/>
-        </visual>
-        <collision>
-            <origin xyz="0.018 0 -0.11" rpy="0 -0.30 0" />
-            <geometry>
-                <box size= "0.02 0.02 0.18"/>
-            </geometry>
-        </collision>
-        <inertial>
-            <origin rpy="0 0 0" xyz="0.0079835 -6.7795E-06 -0.18022"/>
-            <mass value="0.23"/>
-            <inertia ixx="0.002770" ixy="0" ixz="0" iyy="0.002764" iyz="0" izz="0.000041"/>
+        <origin rpy="0 0 0" xyz="0 0 0"/>
+        <geometry>
+            <mesh filename="package://mz_description/meshes/calf.dae" scale="1 1 1"/>
+        </geometry>
+        <material name="silver"/>
+        </visual>
+        <collision>
+        <origin xyz="0.018 0 -0.16" rpy="0 -0.10 0" />
+        <geometry>
+            <box size= "0.02 0.02 0.24"/>
+        </geometry>
+        </collision>
+        <inertial>
+        <origin rpy="0 0 0" xyz="0.01038 0 -0.072"/>
+        <mass value="0.23"/>
+        <inertia ixx="0.009492" ixy="0" ixz="0" iyy="0.009342" iyz="0" izz="0.000366"/>
         </inertial>
     </link>
@@ -388,5 +393,5 @@
         <origin rpy="0 0 0" xyz="0 0 0"/>
         <geometry>
-            <sphere radius="0.025"/>
+            <sphere radius="0.0235"/>
         </geometry>
         </collision>
@@ -400,5 +405,6 @@
     <!-- RL Leg -->
     <joint name="RL_hip_joint" type="revolute">
-        <origin rpy="0 0 0" xyz="-0.22624 0.069992 0.075"/>
+        <!-- trunk com offset is 0.075 -->
+        <origin rpy="0 0 0" xyz="-0.22624 0.07 0.075"/>
         <parent link="trunk"/>
         <child link="RL_hip"/>
@@ -407,16 +413,17 @@
         <limit effort="67" lower="-1.04" upper="1.04" velocity="15"/>
     </joint>
+    <!-- 国庆节修改的hip关节模型 -->
     <link name="RL_hip">
         <visual>
-            <origin xyz="0 0 0" rpy="0 0 0" />
-            <geometry>
-                <mesh filename="package://mz_description/meshes/RL_hip.dae" scale="1 1 1"/>
-            </geometry>
-            <material name="silver"/>
-        </visual>
-        <inertial>
-            <origin rpy="0 0 0" xyz="-0.083541 0.0016537 -1.2994E-05"/>
-            <mass value="1.6"/>
-            <inertia ixx="0.001986561" ixy="0.0" ixz="0.0" iyy="0.002917650" iyz="0.0" izz="0.002219916"/>
+        <origin xyz="0 0 0" rpy="0 0 0" />
+        <geometry>
+            <mesh filename="package://mz_description/meshes/RL_hip.dae" scale="1 1 1"/>
+        </geometry>
+        <material name="silver"/>
+        </visual>
+        <inertial>
+        <origin rpy="0 0 0" xyz="-0.08 0.00177 0.00001"/>
+        <mass value="1.6"/>
+        <inertia ixx="0.001726" ixy="0" ixz="0" iyy="0.003117" iyz="0" izz="0.002200"/>
         </inertial>
     </link>
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