Commit message: 消除了颜色未定义警告

File: src/robots/sz_description/xacro/robot.xacro (robot description, xacro)
@@ -6,4 +6,16 @@
     <xacro:include filename="$(find sz_description)/xacro/transmission.xacro"/>
     <xacro:include filename="$(find sz_description)/xacro/gazebo.xacro"/>
+    <material name="blue">
+        <color rgba="0.0 0.0 0.8 1.0"/>
+    </material>
+    <material name="green">
+        <color rgba="0.0 0.8 0.0 1.0"/>
+    </material>
+    <material name="silver">
+        <color rgba="0.913725490196 0.913725490196 0.847058823529 0.5"/>
+    </material>
+    <material name="red">
+        <color rgba="0.8 0.0 0.0 1.0"/>
+    </material>
     <xacro:if value="$(arg DEBUG)">
         <link name="world"/>

Commit message: 根据实物重新调整sz转动惯量

File: src/robots/sz_description/xacro/robot.xacro (robot description, xacro)
@@ -55,9 +55,22 @@
         <inertial>
         <!-- <origin rpy="0 0 0" xyz="0.012731 0.002186 0.000515"/> -->
-        <origin rpy="0 0 0" xyz="0.038238 -0.0086038 -0.0003117"/>
+        <origin rpy="0 0 0" xyz="0.0 0.0 0.0"/>
         <mass value="5.848"/>
-        <inertia ixx="0.01683993" ixy="8.3902e-05" ixz="0.000597679" iyy="0.056579028" iyz="2.5134e-05" izz="0.064713601"/>
+        <inertia ixx="0.0265" ixy="0.0" ixz="0.0" iyy="0.04660" iyz="0.0" izz="0.05907"/>
         <!-- <inertia ixx="0.01883039838" ixy="-0.00025723812" ixz="-0.00032987281" iyy="0.0705707128" iyz="-0.00004689787" izz="0.0802532948" /> -->
         </inertial>
+    </link>
+    <joint name="head_joint" type="fixed">
+        <parent link="trunk"/>
+        <child link="head"/>
+        <origin rpy="0 0 0" xyz="0.29 0 0"/>
+    </joint>
+    <link name="head">
+        <collision>
+        <origin rpy="0 0 0" xyz="0 0 0"/>
+        <geometry>
+            <box size="0.06 0.13 0.120"/>
+        </geometry>
+        </collision>
     </link>
     <joint name="imu_joint" type="fixed">
@@ -112,5 +125,5 @@
         </collision> -->
         <inertial>
-        <origin rpy="0 0 0" xyz="-0.0037743 0.0038894 7.8535E-05"/>
+        <origin rpy="0 0 0" xyz="0.0037743 -0.0038894 7.8535E-05"/>
         <mass value="0.68"/>
         <inertia ixx="0.000469246" ixy="9.409e-06" ixz="-3.42e-07" iyy="0.00080749" iyz="4.66e-07" izz="0.000552929"/>
@@ -165,5 +178,5 @@
         <origin rpy="0 0 0" xyz="-0.0025418 0.024397 -0.017202"/>
         <mass value="1.009"/>
-        <inertia ixx="0.005529065" ixy="-4.825e-06" ixz="0.000343869" iyy="0.005139339" iyz="-2.2448e-05" izz="0.001367788"/>
+        <inertia ixx="0.006118" ixy="0.0" ixz="0.0" iyy="0.006749" iyz="0.0" izz="0.001051"/>
         <!-- <inertia ixx="0.0059674237094595" ixy="2.463414414414414e-6" ixz="3.941565326576577e-4" iyy="0.0056818460304054" iyz="3.201302477477477e-5" izz="0.0012614772522523" /> -->
         </inertial>
@@ -202,5 +215,5 @@
         <origin rpy="0 0 0" xyz="0.0052583 3.7921E-08 -0.11963"/>
         <mass value="0.224"/>
-        <inertia ixx="0.002997972" ixy="0.0" ixz="-0.000141163" iyy="0.003014022" iyz="0.0" izz="3.2426e-05"/>
+        <inertia ixx="0.001269" ixy="0.0" ixz="0.0" iyy="0.001277" iyz="0.0" izz="0.00002425"/>
         <!-- <inertia ixx="0.0034783165033113" ixy="0.0" ixz="-2.095735099337748e-4" iyy="0.0035020471523179" iyz="0.0" izz="4.622113907284768e-5" /> -->
         </inertial>
@@ -257,7 +270,7 @@
         </collision> -->
         <inertial>
-        <origin rpy="0 0 0" xyz="-0.0037743 0.0038894 7.8535E-05"/>
+        <origin rpy="0 0 0" xyz="0.0037743 0.0038894 7.8535E-05"/>
         <mass value="0.68"/>
-        <inertia ixx="0.000469246" ixy="-9.409e-06" ixz="-3.42e-07" iyy="0.00080749" iyz="-4.66e-07" izz="0.000552929"/>
+        <inertia ixx="0.000469246" ixy="9.409e-06" ixz="-3.42e-07" iyy="0.00080749" iyz="4.66e-07" izz="0.000552929"/>
         <!-- <inertia ixx="4.602822857142857e-4" ixy="-9.953142857142857e-6" ixz="-3.394285714285714e-7" iyy="7.898548571428571e-4" iyz="-6.228571428571429e-7" izz="5.576217142857143e-4" /> -->
         </inertial>
@@ -310,5 +323,5 @@
         <origin rpy="0 0 0" xyz="-0.002926 -0.024388 -0.017656"/>
         <mass value="1.009"/>
-        <inertia ixx="0.005529065" ixy="4.825e-06" ixz="0.000343869" iyy="0.005139339" iyz="2.2448e-05" izz="0.001367788"/>
+        <inertia ixx="0.006118" ixy="0.0" ixz="0.0" iyy="0.006749" iyz="0.0" izz="0.001051"/>
         <!-- <inertia ixx="0.0059674237094595" ixy="-2.463414414414414e-6" ixz="3.941565326576577e-4" iyy="0.0056818460304054" iyz="-3.201302477477477e-5" izz="0.0012614772522523" /> -->
         </inertial>
@@ -346,5 +359,5 @@
         <origin rpy="0 0 0" xyz="0.0052583 3.7881E-08 -0.11963"/>
         <mass value="0.224"/>
-        <inertia ixx="0.002997972" ixy="0.0" ixz="-0.000141163" iyy="0.003014022" iyz="0.0" izz="3.2426e-05"/>
+        <inertia ixx="0.001269" ixy="0.0" ixz="0.0" iyy="0.001277" iyz="0.0" izz="0.00002425"/>
         <!-- <inertia ixx="0.0034783165033113" ixy="0.0" ixz="-2.095735099337748e-4" iyy="0.0035020471523179" iyz="0.0" izz="4.622113907284768e-5" /> -->
         </inertial>
@@ -401,7 +414,7 @@
         </collision> -->
         <inertial>
-        <origin rpy="0 0 0" xyz="0.0037743 0.0038894 -7.8535E-05"/>
+        <origin rpy="0 0 0" xyz="-0.0037743 0.0038894 7.8535E-05"/>
         <mass value="0.68"/>
-        <inertia ixx="0.000469246" ixy="-9.409e-06" ixz="3.42e-07" iyy="0.00080749" iyz="4.66e-07" izz="0.000552929"/>
+        <inertia ixx="0.000469246" ixy="9.409e-06" ixz="-3.42e-07" iyy="0.00080749" iyz="4.66e-07" izz="0.000552929"/>
         <!-- <inertia ixx="4.602822857142857e-4" ixy="-9.953142857142857e-6" ixz="3.394285714285714e-7" iyy="7.898548571428571e-4" iyz="6.228571428571429e-7" izz="5.576217142857143e-4" /> -->
         </inertial>
@@ -454,5 +467,5 @@
         <origin rpy="0 0 0" xyz="-0.0025418 0.024397 -0.017202"/>
         <mass value="1.009"/>
-        <inertia ixx="0.005529065" ixy="-4.825e-06" ixz="0.000343869" iyy="0.005139339" iyz="-2.2448e-05" izz="0.001367788"/>
+        <inertia ixx="0.006118" ixy="0.0" ixz="0.0" iyy="0.006749" iyz="0.0" izz="0.001051"/>
         <!-- <inertia ixx="0.0059674237094595" ixy="2.463414414414414e-6" ixz="3.941565326576577e-4" iyy="0.0056818460304054" iyz="3.201302477477477e-5" izz="0.0012614772522523" /> -->
         </inertial>
@@ -490,5 +503,5 @@
         <origin rpy="0 0 0" xyz="0.0052583 4.9987E-08 -0.11963"/>
         <mass value="0.224"/>
-        <inertia ixx="0.002997972" ixy="0.0" ixz="-0.000141163" iyy="0.003014022" iyz="0.0" izz="3.2426e-05"/>
+        <inertia ixx="0.001269" ixy="0.0" ixz="0.0" iyy="0.001277" iyz="0.0" izz="0.00002425"/>
         <!-- <inertia ixx="0.0034783165033113" ixy="0.0" ixz="-2.095735099337748e-4" iyy="0.0035020471523179" iyz="0.0" izz="4.622113907284768e-5" /> -->
         </inertial>
@@ -545,7 +558,7 @@
         </collision> -->
         <inertial>
-        <origin rpy="0 0 0" xyz="0.0037743 0.0038894 7.8535E-05"/>
+        <origin rpy="0 0 0" xyz="-0.0037743 -0.0038894 7.8535E-05"/>
         <mass value="0.68"/>
-        <inertia ixx="0.000469246" ixy="9.409e-06" ixz="3.42e-07" iyy="0.00080749" iyz="-4.66e-07" izz="0.000552929"/>
+        <inertia ixx="0.000469246" ixy="9.409e-06" ixz="-3.42e-07" iyy="0.00080749" iyz="4.66e-07" izz="0.000552929"/>
         <!-- <inertia ixx="4.602822857142857e-4" ixy="9.953142857142857e-6" ixz="3.394285714285714e-7" iyy="7.898548571428571e-4" iyz="-6.228571428571429e-7" izz="5.576217142857143e-4" /> -->
         </inertial>
@@ -598,5 +611,5 @@
         <origin rpy="0 0 0" xyz="-0.002926 -0.024388 -0.017656"/>
         <mass value="1.009"/>
-        <inertia ixx="0.005529065" ixy="4.825e-06" ixz="0.000343869" iyy="0.005139339" iyz="2.2448e-05" izz="0.001367788"/>
+        <inertia ixx="0.006118" ixy="0.0" ixz="0.0" iyy="0.006749" iyz="0.0" izz="0.001051"/>
         <!-- <inertia ixx="0.0059674237094595" ixy="-2.463414414414414e-6" ixz="3.941565326576577e-4" iyy="0.0056818460304054" iyz="-3.201302477477477e-5" izz="0.0012614772522523" /> -->
         </inertial>
@@ -634,5 +647,5 @@
         <origin rpy="0 0 0" xyz="0.0052583 3.799E-08 -0.11963"/>
         <mass value="0.224"/>
-        <inertia ixx="0.002997972" ixy="0.0" ixz="-0.000141163" iyy="0.003014022" iyz="0.0" izz="3.2426e-05"/>
+        <inertia ixx="0.001269" ixy="0.0" ixz="0.0" iyy="0.001277" iyz="0.0" izz="0.00002425"/>
         <!-- <inertia ixx="0.0034783165033113" ixy="0.0" ixz="-1.614571428571429e-4" iyy="0.0026824344538288" iyz="0.0" izz="3.540362837837838e-5" /> -->
         </inertial>
@@ -654,5 +667,5 @@
         <origin rpy="0 0 0" xyz="0 0 0"/>
         <geometry>
-            <sphere radius="0.02"/>
+            <sphere radius="0.025"/>
         </geometry>
         </collision>

Commit message: 修正小型四足机器人urdf模型中hip关节的质心位置

File: src/robots/sz_description/xacro/robot.xacro (robot description, xacro)
@@ -414,5 +414,5 @@
         </collision> -->
         <inertial>
-        <origin rpy="0 0 0" xyz="-0.0037743 0.0038894 7.8535E-05"/>
+        <origin rpy="0 0 0" xyz="-0.0037743 -0.0038894 7.8535E-05"/>
         <mass value="0.68"/>
         <inertia ixx="0.000469246" ixy="9.409e-06" ixz="-3.42e-07" iyy="0.00080749" iyz="4.66e-07" izz="0.000552929"/>
@@ -558,5 +558,5 @@
         </collision> -->
         <inertial>
-        <origin rpy="0 0 0" xyz="-0.0037743 -0.0038894 7.8535E-05"/>
+        <origin rpy="0 0 0" xyz="-0.0037743 0.0038894 7.8535E-05"/>
         <mass value="0.68"/>
         <inertia ixx="0.000469246" ixy="9.409e-06" ixz="-3.42e-07" iyy="0.00080749" iyz="4.66e-07" izz="0.000552929"/>

Commit message: 将小型四足机器人urdf模型hip关节的惯量积置零

File: src/robots/sz_description/xacro/robot.xacro (robot description, xacro)
@@ -127,5 +127,5 @@
         <origin rpy="0 0 0" xyz="0.0037743 -0.0038894 7.8535E-05"/>
         <mass value="0.68"/>
-        <inertia ixx="0.000469246" ixy="9.409e-06" ixz="-3.42e-07" iyy="0.00080749" iyz="4.66e-07" izz="0.000552929"/>
+        <inertia ixx="0.000469246" ixy="0.0" ixz="0.0" iyy="0.00080749" iyz="0.0" izz="0.000552929"/>
         <!-- <inertia ixx="4.602822857142857e-4" ixy="9.953142857142857e-6" ixz="-3.394285714285714e-7" iyy="7.898548571428571e-4" iyz="6.228571428571429e-7" izz="5.576217142857143e-4" /> -->
         </inertial>
@@ -272,5 +272,5 @@
         <origin rpy="0 0 0" xyz="0.0037743 0.0038894 7.8535E-05"/>
         <mass value="0.68"/>
-        <inertia ixx="0.000469246" ixy="9.409e-06" ixz="-3.42e-07" iyy="0.00080749" iyz="4.66e-07" izz="0.000552929"/>
+        <inertia ixx="0.000469246" ixy="0.0" ixz="0.0" iyy="0.00080749" iyz="0.0" izz="0.000552929"/>
         <!-- <inertia ixx="4.602822857142857e-4" ixy="-9.953142857142857e-6" ixz="-3.394285714285714e-7" iyy="7.898548571428571e-4" iyz="-6.228571428571429e-7" izz="5.576217142857143e-4" /> -->
         </inertial>
@@ -416,5 +416,5 @@
         <origin rpy="0 0 0" xyz="-0.0037743 -0.0038894 7.8535E-05"/>
         <mass value="0.68"/>
-        <inertia ixx="0.000469246" ixy="9.409e-06" ixz="-3.42e-07" iyy="0.00080749" iyz="4.66e-07" izz="0.000552929"/>
+        <inertia ixx="0.000469246" ixy="0.0" ixz="0.0" iyy="0.00080749" iyz="0.0" izz="0.000552929"/>
         <!-- <inertia ixx="4.602822857142857e-4" ixy="-9.953142857142857e-6" ixz="3.394285714285714e-7" iyy="7.898548571428571e-4" iyz="6.228571428571429e-7" izz="5.576217142857143e-4" /> -->
         </inertial>
@@ -560,5 +560,5 @@
         <origin rpy="0 0 0" xyz="-0.0037743 0.0038894 7.8535E-05"/>
         <mass value="0.68"/>
-        <inertia ixx="0.000469246" ixy="9.409e-06" ixz="-3.42e-07" iyy="0.00080749" iyz="4.66e-07" izz="0.000552929"/>
+        <inertia ixx="0.000469246" ixy="0.0" ixz="0.0" iyy="0.00080749" iyz="0.0" izz="0.000552929"/>
         <!-- <inertia ixx="4.602822857142857e-4" ixy="9.953142857142857e-6" ixz="3.394285714285714e-7" iyy="7.898548571428571e-4" iyz="-6.228571428571429e-7" izz="5.576217142857143e-4" /> -->
         </inertial>
