Commit message: 人形机器人仿真环境搭建完成

File: src/robots/gh1_description/urdf/gh1_description.urdf (robot description, URDF)
Before this commit: robot gh1_description, 21 links, 20 joints
Links:
- removed link Left_elbow_pitch_Link
- removed link Left_shoulder_pitch_Link
- removed link Left_shoulder_roll_Link
- removed link Left_shoulder_yaw_Link
- removed link Right_elbow_pitch_Link
- removed link Right_shoulder_pitch_Link
- removed link Right_shoulder_roll_Link
- removed link Right_shoulder_yaw_Link
- link Left_ankle_pitch_Link: mass 0.38818 -> 0.27473; geometry collision box size=0.25 0.05 0.02; visual mesh filename=package://gh1_description/meshes/L5_link.STL
- link Left_hip_pitch_Link: mass 33.931 -> 1.2137; geometry collision box size=0.07 0.05 0.35; visual mesh filename=package://gh1_description/meshes/L3_link.STL
- link Left_hip_roll_Link: mass 3.8235 -> 0.76576; geometry collision cylinder length=0.06 radius=0.06; visual mesh filename=package://gh1_description/meshes/L1_link.STL
- link Left_hip_yaw_Link: mass 6.7642 -> 0.68726; geometry collision cylinder length=0.15 radius=0.06; visual mesh filename=package://gh1_description/meshes/L2_link.STL
- link Left_knee_Link: mass 7.7671 -> 0.70946; geometry collision box size=0.06 0.029 0.32; visual mesh filename=package://gh1_description/meshes/L4_link.STL
- link Right_ankle_pitch_Link: mass 0.38818 -> 0.27473; geometry collision box size=0.25 0.05 0.02; visual mesh filename=package://gh1_description/meshes/R5_link.STL
- link Right_hip_pitch_Link: mass 33.93 -> 1.2137; geometry collision box size=0.07 0.05 0.35; visual mesh filename=package://gh1_description/meshes/R3_link.STL
- link Right_hip_roll_Link: mass 3.7336 -> 0.76576; geometry collision cylinder length=0.06 radius=0.06; visual mesh filename=package://gh1_description/meshes/R1_link.STL
- link Right_hip_yaw_Link: mass 6.9007 -> 0.68726; geometry collision cylinder length=0.15 radius=0.06; visual mesh filename=package://gh1_description/meshes/R2_link.STL
- link Right_knee_Link: mass 7.7671 -> 0.70946; geometry collision box size=0.06 0.029 0.32; visual mesh filename=package://gh1_description/meshes/R4_link.STL
- link body: mass 123.52 -> 10.935; geometry collision box size=0.18 0.28 0.4; collision cylinder length=0.28 radius=0.01
Joints:
- removed joint Left_ankle_pitch_Joint
- removed joint Left_elbow_pitch_Joint
- removed joint Left_hip_pitch_Joint
- removed joint Left_hip_roll_Joint
- removed joint Left_hip_yaw_Joint
- removed joint Left_knee_Joint
- removed joint Left_shoulder_pitch_Joint
- removed joint Left_shoulder_roll_Joint
- removed joint Left_shoulder_yaw_Joint
- removed joint Right_ankle_pitch_Joint
- removed joint Right_elbow_pitch_Joint
- removed joint Right_hip_pitch_Joint
- removed joint Right_hip_roll_Joint
- removed joint Right_hip_yaw_Joint
- removed joint Right_knee_Joint
- removed joint Right_shoulder_pitch_Joint
- removed joint Right_shoulder_roll_Joint
- removed joint Right_shoulder_yaw_Joint
- added joint l_ankle_pitch: type revolute, parent Left_knee_Link, child Left_ankle_pitch_Link, origin xyz=0 0 -0.4 rpy=0 0 0, axis 0 1 0, limit lower=-1.08 upper=0.59 effort=22 velocity=46.024
- added joint l_hip_pitch: type revolute, parent Left_hip_yaw_Link, child Left_hip_pitch_Link, origin xyz=0 -0.041 -0.127 rpy=0 0 0, axis 0 1 0, limit lower=-1.75 upper=1.75 effort=120 velocity=20.92
- added joint l_hip_roll: type revolute, parent body, child Left_hip_roll_Link, origin xyz=-0.08275 0.135 -0.2975 rpy=0 0 0, axis 1 0 0, limit lower=-0.17 upper=1.05 effort=120 velocity=20.92
- added joint l_hip_yaw: type revolute, parent Left_hip_roll_Link, child Left_hip_yaw_Link, origin xyz=0.087 0 -0.015 rpy=0 0 0, axis 0 0 1, limit lower=-1.66 upper=1.66 effort=70 velocity=12.552
- added joint l_knee_pitch: type revolute, parent Left_hip_pitch_Link, child Left_knee_Link, origin xyz=0 0.041 -0.42 rpy=0 0 0, axis 0 1 0, limit lower=0.56 upper=2.23 effort=120 velocity=20.92
- added joint r_ankle_pitch: type revolute, parent Right_knee_Link, child Right_ankle_pitch_Link, origin xyz=0 0 -0.4 rpy=0 0 0, axis 0 1 0, limit lower=-1.08 upper=0.59 effort=22 velocity=46.024
- added joint r_hip_pitch: type revolute, parent Right_hip_yaw_Link, child Right_hip_pitch_Link, origin xyz=0 0.041 -0.127 rpy=0 0 0, axis 0 1 0, limit lower=-1.75 upper=1.75 effort=120 velocity=20.92
- added joint r_hip_roll: type revolute, parent body, child Right_hip_roll_Link, origin xyz=-0.08275 -0.135 -0.2975 rpy=0 0 0, axis 1 0 0, limit lower=-1.05 upper=0.17 effort=120 velocity=20.92
- added joint r_hip_yaw: type revolute, parent Right_hip_roll_Link, child Right_hip_yaw_Link, origin xyz=0.087 0 -0.015 rpy=0 0 0, axis 0 0 1, limit lower=-1.66 upper=1.66 effort=70 velocity=12.552
- added joint r_knee_pitch: type revolute, parent Right_hip_pitch_Link, child Right_knee_Link, origin xyz=0 -0.041 -0.42 rpy=0 0 0, axis 0 1 0, limit lower=0.56 upper=2.23 effort=120 velocity=20.92
- joint z_joint_imu: origin xyz=-0.0648 0 -0.1015 rpy=0 0 0 -> xyz=-0.0 0 -0.0 rpy=0 0 0

Commit message: 修改了质量惯量，将连杆的名称与宇树对应

File: src/robots/gh1_description/urdf/gh1_description.urdf (robot description, URDF)
Before this commit: robot gh1_description, 13 links, 12 joints
Links:
- removed link Left_ankle_pitch_Link
- removed link Left_hip_pitch_Link
- removed link Left_hip_roll_Link
- removed link Left_hip_yaw_Link
- removed link Left_knee_Link
- removed link Right_ankle_pitch_Link
- removed link Right_hip_pitch_Link
- removed link Right_hip_roll_Link
- removed link Right_hip_yaw_Link
- removed link Right_knee_Link
- added link l_foot_pitch, mass 0.55; collision box size=0.25 0.05 0.02; visual mesh filename=package://gh1_description/meshes/L5_link.STL
- added link l_shank_pitch, mass 1.88; collision box size=0.06 0.029 0.32; visual mesh filename=package://gh1_description/meshes/L4_link.STL
- added link l_thigh_pitch, mass 4.07; collision box size=0.07 0.05 0.35; visual mesh filename=package://gh1_description/meshes/L3_link.STL
- added link l_thigh_roll, mass 2.19; collision cylinder length=0.06 radius=0.06; visual mesh filename=package://gh1_description/meshes/L1_link.STL
- added link l_thigh_yaw, mass 2.72; collision cylinder length=0.15 radius=0.06; visual mesh filename=package://gh1_description/meshes/L2_link.STL
- added link r_foot_pitch, mass 0.55; collision box size=0.25 0.05 0.02; visual mesh filename=package://gh1_description/meshes/R5_link.STL
- added link r_shank_pitch, mass 1.88; collision box size=0.06 0.029 0.32; visual mesh filename=package://gh1_description/meshes/R4_link.STL
- added link r_thigh_pitch, mass 4.07; collision box size=0.07 0.05 0.35; visual mesh filename=package://gh1_description/meshes/R3_link.STL
- added link r_thigh_roll, mass 2.19; collision cylinder length=0.06 radius=0.06; visual mesh filename=package://gh1_description/meshes/R1_link.STL
- added link r_thigh_yaw, mass 2.72; collision cylinder length=0.15 radius=0.06; visual mesh filename=package://gh1_description/meshes/R2_link.STL
Joints:
- joint l_ankle_pitch: child Left_ankle_pitch_Link -> l_foot_pitch; parent Left_knee_Link -> l_shank_pitch
- joint l_hip_pitch: child Left_hip_pitch_Link -> l_thigh_pitch; parent Left_hip_yaw_Link -> l_thigh_yaw
- joint l_hip_roll: child Left_hip_roll_Link -> l_thigh_roll
- joint l_hip_yaw: child Left_hip_yaw_Link -> l_thigh_yaw; parent Left_hip_roll_Link -> l_thigh_roll
- joint l_knee_pitch: child Left_knee_Link -> l_shank_pitch; parent Left_hip_pitch_Link -> l_thigh_pitch
- joint r_ankle_pitch: child Right_ankle_pitch_Link -> r_foot_pitch; parent Right_knee_Link -> r_shank_pitch
- joint r_hip_pitch: child Right_hip_pitch_Link -> r_thigh_pitch; parent Right_hip_yaw_Link -> r_thigh_yaw
- joint r_hip_roll: child Right_hip_roll_Link -> r_thigh_roll
- joint r_hip_yaw: child Right_hip_yaw_Link -> r_thigh_yaw; parent Right_hip_roll_Link -> r_thigh_roll
- joint r_knee_pitch: child Right_knee_Link -> r_shank_pitch; parent Right_hip_pitch_Link -> r_thigh_pitch

Commit message: 将人形机器人的body默认固定在空中,通过注释gh1_description.urdf中的base_static_joint来取消悬浮

File: src/robots/gh1_description/urdf/gh1_description.urdf (robot description, URDF)
Before this commit: robot gh1_description, 13 links, 12 joints
Links:
- added link world
Joints:
- added joint base_static_joint: type fixed, parent world, child base, origin xyz=0 0 -0.5 rpy=0 0 0

File: src/robots/gh1_description/xacro/robot.xacro (robot description, xacro)
@@ -13,5 +13,5 @@
     <link name="world" />
     <joint name="base_static_joint" type="fixed">
-      <origin rpy="0 0 0" xyz="0 0 0" />
+      <origin rpy="0 0 0" xyz="0 0 1.6" />
       <parent link="world" />
       <child link="base" />
