Commit message: 将gazebo_gh.launch默认启动xacro文件,将urdf内容迁移至robot.xacro文件中,后续还需要将gr1t1的urdf中的内容迁移至xacro中,目前无该需求

File: src/robots/gh1_description/xacro/gazebo.xacro (robot description, xacro)
@@ -1,36 +1,153 @@
 <?xml version="1.0"?>
 <robot>
-    <!-- ros_control plugin -->
-    <gazebo>
-        <plugin name="gazebo_ros_control" filename="libgazebo_ros_control.so">
-            <robotNamespace>/g1_gazebo</robotNamespace>
-            <robotSimType>gazebo_ros_control/DefaultRobotHWSim</robotSimType>
+  <gazebo>
+    <plugin filename="libgazebo_ros_control.so" name="gazebo_ros_control">
+      <robotNamespace>/gh1_gazebo</robotNamespace>
+      <robotSimType>gazebo_ros_control/DefaultRobotHWSim</robotSimType>
+    </plugin>
+  </gazebo>
+  <!-- Show the trajectory of base_link center. -->
+  <!-- <gazebo>
+        <plugin name="3dplot" filename="libLinkPlot3DPlugin.so">
+            <frequency>10</frequency>
+            <plot>
+                <link>base</link>
+                <pose>0 0 0 0 0 0</pose>
+                <material>Gazebo/Yellow</material>
+            </plot>
         </plugin>
-    </gazebo>
-    <gazebo reference="imu_link">
-        <gravity>true</gravity>
-        <sensor name="imu_sensor" type="imu">
-            <always_on>true</always_on>
-            <update_rate>1000</update_rate>
-            <visualize>true</visualize>
-            <topic>__default_topic__</topic>
-            <plugin filename="libgazebo_ros_imu_sensor.so" name="imu_plugin">
-                <topicName>trunk_imu</topicName>
-                <bodyName>imu_link</bodyName>
-                <updateRateHZ>1000.0</updateRateHZ>
-                <gaussianNoise>0.0</gaussianNoise>
-                <xyzOffset>0 0 0</xyzOffset>
-                <rpyOffset>0 0 0</rpyOffset>
-                <frameName>imu_link</frameName>
-            </plugin>
-            <pose>0 0 0 0 0 0</pose>
-        </sensor>
-    </gazebo>
-    <gazebo reference="base">
-        <turnGravityOff>false</turnGravityOff>
-    </gazebo>
-    <gazebo reference="imu_link">
-        <mu1>0.2</mu1>
-        <mu2>0.2</mu2>
-    </gazebo>
+    </gazebo> -->
+  <!-- Show the trajectory of foot. You can add another trajectory about another foot. -->
+  <!-- <gazebo>
+        <plugin name="3dplot" filename="libLinkPlot3DPlugin.so">
+            <frequency>100</frequency>
+            <plot>
+                <link>FL_foot</link>
+                <pose>0 0 0 0 0 0</pose>
+                <material>Gazebo/Green</material>
+            </plot>
+        </plugin>
+    </gazebo> -->
+  <gazebo>
+    <plugin filename="libgazebo_ros_force.so" name="gazebo_ros_force">
+      <bodyName>body</bodyName>
+      <topicName>/apply_force/body</topicName>
+    </plugin>
+  </gazebo>
+  <gazebo reference="imu_link">
+    <gravity>true</gravity>
+    <sensor name="imu_sensor" type="imu">
+      <always_on>true</always_on>
+      <update_rate>1000</update_rate>
+      <visualize>true</visualize>
+      <topic>__default_topic__</topic>
+      <plugin filename="libgazebo_ros_imu_sensor.so" name="imu_plugin">
+        <topicName>base_link_imu</topicName>
+        <bodyName>imu_link</bodyName>
+        <updateRateHZ>1000.0</updateRateHZ>
+        <gaussianNoise>0.0</gaussianNoise>
+        <xyzOffset>0 0 0</xyzOffset>
+        <rpyOffset>0 0 0</rpyOffset>
+        <frameName>imu_link</frameName>
+      </plugin>
+      <pose>0 0 0 0 0 0</pose>
+    </sensor>
+  </gazebo>
+  <gazebo reference="base">
+    <material>Gazebo/DarkGrey</material>
+    <turnGravityOff>false</turnGravityOff>
+  </gazebo>
+  <gazebo reference="body">
+    <mu1>0.2</mu1>
+    <mu2>0.2</mu2>
+    <kp value="1000000.0" />
+    <kd value="1.0" />
+  </gazebo>
+  <gazebo reference="imu_link">
+    <mu1>0.2</mu1>
+    <mu2>0.2</mu2>
+    <material>Gazebo/Red</material>
+  </gazebo>
+  <!-- left leg -->
+  <gazebo reference="l_thigh_roll">
+    <mu1>0.2</mu1>
+    <mu2>0.2</mu2>
+    <self_collide>1</self_collide>
+    <material>Gazebo/DarkGrey</material>
+  </gazebo>
+  <gazebo reference="l_thigh_yaw">
+    <mu1>0.2</mu1>
+    <mu2>0.2</mu2>
+    <self_collide>1</self_collide>
+    <material>Gazebo/DarkGrey</material>
+  </gazebo>
+  <gazebo reference="l_thigh_pitch">
+    <mu1>0.2</mu1>
+    <mu2>0.2</mu2>
+    <self_collide>1</self_collide>
+    <material>Gazebo/DarkGrey</material>
+  </gazebo>
+  <gazebo reference="l_shank_pitch">
+    <mu1>0.2</mu1>
+    <mu2>0.2</mu2>
+    <self_collide>1</self_collide>
+    <material>Gazebo/DarkGrey</material>
+  </gazebo>
+  <gazebo reference="l_foot_pitch">
+    <mu1>1.0</mu1>
+    <mu2>1.0</mu2>
+    <self_collide>1</self_collide>
+    <kp value="1000000.0" />
+    <kd value="1.0" />
+    <material>Gazebo/DarkGrey</material>
+  </gazebo>
+  <gazebo reference="l_foot_roll">
+    <mu1>1.0</mu1>
+    <mu2>1.0</mu2>
+    <self_collide>1</self_collide>
+    <kp value="1000000.0" />
+    <kd value="1.0" />
+    <material>Gazebo/DarkGrey</material>
+  </gazebo>
+  <!-- right leg -->
+  <gazebo reference="r_thigh_roll">
+    <mu1>0.2</mu1>
+    <mu2>0.2</mu2>
+    <self_collide>1</self_collide>
+    <material>Gazebo/DarkGrey</material>
+  </gazebo>
+  <gazebo reference="r_thigh_yaw">
+    <mu1>0.2</mu1>
+    <mu2>0.2</mu2>
+    <self_collide>1</self_collide>
+    <material>Gazebo/DarkGrey</material>
+  </gazebo>
+  <gazebo reference="r_thigh_pitch">
+    <mu1>0.2</mu1>
+    <mu2>0.2</mu2>
+    <self_collide>1</self_collide>
+    <material>Gazebo/DarkGrey</material>
+  </gazebo>
+  <gazebo reference="r_shank_pitch">
+    <mu1>0.2</mu1>
+    <mu2>0.2</mu2>
+    <self_collide>1</self_collide>
+    <material>Gazebo/DarkGrey</material>
+  </gazebo>
+  <gazebo reference="r_foot_pitch">
+    <mu1>1.0</mu1>
+    <mu2>1.0</mu2>
+    <self_collide>1</self_collide>
+    <kp value="1000000.0" />
+    <kd value="1.0" />
+    <material>Gazebo/DarkGrey</material>
+  </gazebo>
+  <gazebo reference="r_foot_roll">
+    <mu1>1.0</mu1>
+    <mu2>1.0</mu2>
+    <self_collide>1</self_collide>
+    <kp value="1000000.0" />
+    <kd value="1.0" />
+    <material>Gazebo/DarkGrey</material>
+  </gazebo>
 </robot>

File: src/robots/gh1_description/xacro/robot.xacro (robot description, xacro)
@@ -3,15 +3,39 @@
   <xacro:arg name="DEBUG" default="false" />
   <xacro:include filename="$(find gh1_description)/xacro/gazebo.xacro" />
-  <xacro:include filename="$(find gh1_description)/xacro/const.xacro" />
-  <xacro:include filename="$(find gh1_description)/xacro/leg.xacro" />
-  <xacro:include filename="$(find gh1_description)/xacro/arm.xacro" />
   <!-- Rotor related joint and link is only for demonstrate location. -->
   <!-- Actually, the rotor will rotate and the joint is not fixed. Reduction ratio should be
   considered. -->
+  <material name="black">
+    <color rgba="0.0 0.0 0.0 1.0" />
+  </material>
+  <material name="blue">
+    <color rgba="0.0 0.0 0.8 1.0" />
+  </material>
+  <material name="green">
+    <color rgba="0.0 0.8 0.0 1.0" />
+  </material>
+  <material name="grey">
+    <color rgba="0.2 0.2 0.2 1.0" />
+  </material>
+  <material name="silver">
+    <color rgba="0.913725490196 0.913725490196 0.847058823529 1.0" />
+  </material>
+  <material name="orange">
+    <color rgba="0.12 0.15 0.2 1.0" />
+  </material>
+  <material name="brown">
+    <color rgba="0.870588235294 0.811764705882 0.764705882353 1.0" />
+  </material>
+  <material name="red">
+    <color rgba="0.8 0.0 0.0 1.0" />
+  </material>
+  <material name="white">
+    <color rgba="1.0 1.0 1.0 1.0" />
+  </material>
   <!-- Debug mode will hung up the robot, use "true" or "false" to switch it. -->
   <xacro:if value="$(arg DEBUG)">
     <link name="world" />
     <joint name="base_static_joint" type="fixed">
-      <origin rpy="0 0 0" xyz="0 0 1.6" />
+      <origin rpy="0 0 0" xyz="0 0 -0.5" />
       <parent link="world" />
       <child link="base" />
@@ -31,16 +55,84 @@
     <child link="body" />
   </joint>
-  <!-- Torso -->
   <link name="body">
     <inertial>
-      <origin xyz="-0.0088989 -1.3208E-07 0.16344" rpy="0 0 0" />
-      <mass value="123.52" />
-      <inertia ixx="1.6862" ixy="1.545E-07" ixz="-5.5846E-05" iyy="1.1047" iyz="1.791E-06"
-        izz="0.89583" />
-    </inertial>
-    <visual>
-      <origin xyz="0 0 0" rpy="0 0 0" />
-      <geometry>
-        <mesh filename="package://gh1_description/meshes/body.dae" />
+      <origin
+        xyz="-0.0057915 -8.0007E-06 -0.045258"
+        rpy="0 0 0" />
+      <mass
+        value="10.935" />
+      <inertia
+        ixx="0.12979"
+        ixy="1.4382E-06"
+        ixz="-0.00016277"
+        iyy="0.099343"
+        iyz="-2.2433E-07"
+        izz="0.067516" />
+    </inertial>
+    <visual>
+      <origin
+        xyz="0 0 0"
+        rpy="0 0 0" />
+      <geometry>
+        <mesh
+          filename="package://gh1_description/meshes/base_link.STL" />
+      </geometry>
+      <material
+        name="">
+        <color
+          rgba="1 1 1 0.3" />
+      </material>
+    </visual>
+    <!-- trunk -->
+    <collision>
+      <origin
+        xyz="0 0 0"
+        rpy="0 0 0" />
+      <geometry>
+        <box size="0.18 0.28 0.4" />
+      </geometry>
+    </collision>
+    <!-- upper right arm -->
+    <collision>
+      <origin
+        xyz="0 -0.24 0"
+        rpy="-0.15 0 0" />
+      <geometry>
+        <cylinder radius="0.01" length="0.28" />
+      </geometry>
+    </collision>
+    <!-- upper left arm -->
+    <collision>
+      <origin
+        xyz="0 0.24 0"
+        rpy="0.15 0 0" />
+      <geometry>
+        <cylinder radius="0.01" length="0.28" />
+      </geometry>
+    </collision>
+    <!-- lower right arm -->
+    <collision>
+      <origin
+        xyz="0.06 -0.3 -0.3"
+        rpy="-0.3 -0.45 0" />
+      <geometry>
+        <cylinder radius="0.01" length="0.28" />
+      </geometry>
+    </collision>
+    <!-- lower left arm -->
+    <collision>
+      <origin
+        xyz="0.06 0.3 -0.3"
+        rpy="0.3 -0.45 0" />
+      <geometry>
+        <cylinder radius="0.01" length="0.28" />
+      </geometry>
+    </collision>
+  </link>
+  <link name="imu_link">
+    <visual>
+      <origin xyz="-0.0 0 -0.0" rpy="0 0 0" />
+      <geometry>
+        <box size="0.05 0.05 0.02" />
       </geometry>
       <material name="">
@@ -48,50 +140,649 @@
       </material>
     </visual>
-    <collision>
-      <origin xyz="0 0 0.175" rpy="0 0 0" />
-      <geometry> <!-- <mesh filename="package://gh1_description/meshes/body.STL" /> -->
-        <box size="0.130 0.3 0.35" />
-      </geometry>
-    </collision>
-  </link>
-  <joint name="imu_joint" type="fixed">
-    <origin xyz="-0.04233868314 0.00166 0.152067" rpy="0 0 0" />
+  </link>
+  <joint name="z_joint_imu" type="fixed">
+    <origin xyz="-0.0 0 -0.0" rpy="0 0 0" />
     <parent link="body" />
     <child link="imu_link" />
   </joint>
-  <!-- IMU -->
-  <link name="imu_link">
-    <inertial>
-      <mass value="0.001" />
-      <origin rpy="0 0 0" xyz="0 0 0" />
-      <inertia ixx="0.0001" ixy="0" ixz="0" iyy="0.0001" iyz="0" izz="0.0001" />
-    </inertial>
-    <visual>
-      <origin rpy="0 0 0" xyz="0 0 0" />
-      <geometry>
-        <box size="0.001 0.001 0.001" />
-      </geometry>
-      <!-- <material name="red"/> -->
-    </visual>
-    <collision>
-      <origin rpy="0 0 0" xyz="0 0 0" />
-      <geometry>
-        <box size=".001 .001 .001" />
-      </geometry>
-    </collision>
-  </link>
-  <!-- <xacro:leg name="left" mirror="1" />
-  <xacro:leg name="right" mirror="-1" />
-  <xacro:arm name="left" mirror="1" />
-  <xacro:arm name="right" mirror="-1" /> -->
-  <!-- <transmission name="torso_tran">
-    <type>transmission_interface/SimpleTransmission</type>
-    <joint name="torso_joint">
-      <hardwareInterface>hardware_interface/EffortJointInterface</hardwareInterface>
-    </joint>
-    <actuator name="torso_motor">
-      <hardwareInterface>hardware_interface/EffortJointInterface</hardwareInterface>
-      <mechanicalReduction>1</mechanicalReduction>
-    </actuator>
-  </transmission> -->
+  <link
+    name="l_thigh_roll">
+    <inertial>
+      <origin
+        xyz="0.078159 0.0 0.003801"
+        rpy="0 0 0" />
+      <mass
+        value="2.19" />
+      <inertia
+        ixx="0.00262800"
+        ixy="0"
+        ixz="0"
+        iyy="0.00262800"
+        iyz="0"
+        izz="0.00394200" />
+    </inertial>
+    <visual>
+      <origin
+        xyz="0 0 0"
+        rpy="0 0 0" />
+      <geometry>
+        <mesh
+          filename="package://gh1_description/meshes/L1_link.STL" />
+      </geometry>
+      <material
+        name="">
+        <color
+          rgba="1 1 1 0.3" />
+      </material>
+    </visual>
+    <collision>
+      <origin
+        xyz="0.085 0 0"
+        rpy="0 0 0" />
+      <geometry>
+        <cylinder radius="0.06" length="0.06" />
+      </geometry>
+    </collision>
+  </link>
+  <joint
+    name="l_hip_roll"
+    type="revolute">
+    <origin
+      xyz="-0.08275 0.135 -0.2975"
+      rpy="0 0 0" />
+    <parent
+      link="body" />
+    <child
+      link="l_thigh_roll" />
+    <axis
+      xyz="1 0 0" />
+    <dynamics damping="0.1" friction="0.2"/>
+    <limit
+      lower="-0.17"
+      upper="1.05"
+      effort="120"
+      velocity="20.92" />
+  </joint>
+  <link
+    name="l_thigh_yaw">
+    <inertial>
+      <origin
+        xyz="-1.5406E-05 -0.039347 -0.093587"
+        rpy="0 0 0" />
+      <mass
+        value="2.72" />
+      <inertia
+        ixx="0.00754800"
+        ixy="0"
+        ixz="0"
+        iyy="0.00754800"
+        iyz="0"
+        izz="0.00489600" />
+    </inertial>
+    <visual>
+      <origin
+        xyz="0 0 0"
+        rpy="0 0 0" />
+      <geometry>
+        <mesh
+          filename="package://gh1_description/meshes/L2_link.STL" />
+      </geometry>
+      <material
+        name="">
+        <color
+          rgba="1 1 1 0.3" />
+      </material>
+    </visual>
+    <collision>
+      <origin
+        xyz="0 -0.01 -0.13"
+        rpy="-1.57 0 0" />
+      <geometry>
+        <cylinder radius="0.06" length="0.15" />
+      </geometry>
+    </collision>
+  </link>
+  <joint
+    name="l_hip_yaw"
+    type="revolute">
+    <origin
+      xyz="0.087 0 -0.015"
+      rpy="0 0 0" />
+    <parent link="l_thigh_roll" />
+    <child link="l_thigh_yaw" />
+    <axis
+      xyz="0 0 1" />
+    <dynamics damping="0.1" friction="0.2"/>
+    <limit
+      lower="-1.66"
+      upper="1.66"
+      effort="70"
+      velocity="12.552" />
+  </joint>
+  <link name="l_thigh_pitch">
+    <inertial>
+      <origin
+        xyz="0.0075478 0.052643 -0.12044"
+        rpy="0 0 0" />
+      <mass
+        value="4.07" />
+      <inertia
+        ixx="0.04239583"
+        ixy="0"
+        ixz="0"
+        iyy="0.04320983"
+        iyz="0"
+        izz="0.00250983" />
+    </inertial>
+    <visual>
+      <origin
+        xyz="0 0 0"
+        rpy="0 0 0" />
+      <geometry>
+        <mesh
+          filename="package://gh1_description/meshes/L3_link.STL" />
+      </geometry>
+      <material
+        name="">
+        <color
+          rgba="1 1 1 0.3" />
+      </material>
+    </visual>
+    <collision>
+      <origin
+        xyz="0.02 0.04 -0.25"
+        rpy="0 0 0" />
+      <geometry>
+        <box size="0.07 0.05 0.35"/>
+      </geometry>
+    </collision>
+  </link>
+  <joint name="l_hip_pitch" type="revolute">
+    <origin
+      xyz="0 -0.041 -0.127"
+      rpy="0 0 0" />
+    <parent link="l_thigh_yaw" />
+    <child link="l_thigh_pitch" />
+    <axis
+      xyz="0 1 0" />
+    <dynamics damping="0.1" friction="0.2"/>
+    <limit
+      lower="-1.75"
+      upper="1.75"
+      effort="120"
+      velocity="20.92" />
+  </joint>
+  <link name="l_shank_pitch">
+    <inertial>
+      <origin
+        xyz="0.0023769 -0.0025816 -0.15422"
+        rpy="0 0 0" />
+      <mass
+        value="1.88" />
+      <inertia
+        ixx="0.01617442"
+        ixy="0"
+        ixz="0"
+        iyy="0.01660667"
+        iyz="0"
+        izz="0.00069576" />
+    </inertial>
+    <visual>
+      <origin
+        xyz="0 0 0"
+        rpy="0 0 0" />
+      <geometry>
+        <mesh
+          filename="package://gh1_description/meshes/L4_link.STL" />
+      </geometry>
+      <material
+        name="">
+        <color
+          rgba="1 1 1 0.3" />
+      </material>
+    </visual>
+    <collision>
+      <origin
+        xyz="0 0 -0.22"
+        rpy="0 0 0" />
+      <geometry>
+        <box size="0.06 0.029 0.32"/>
+      </geometry>
+    </collision>
+  </link>
+  <joint name="l_knee_pitch" type="revolute">
+    <origin
+      xyz="0 0.041 -0.42"
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