Commit message: 将gr1t1的urdf中的内容迁移至xacro文件中,存在启动gh1导致模型加载出错出现大方块的bug(偶尔出现)

File: src/robots/gh1_description/xacro/robot.xacro (robot description, xacro)
@@ -197,5 +197,5 @@
     <axis
       xyz="1 0 0" />
-    <dynamics damping="0.1" friction="0.2"/>
+    <dynamics damping="0.03" friction="0.2"/>
     <limit
       lower="-0.17"
@@ -253,5 +253,5 @@
     <axis
       xyz="0 0 1" />
-    <dynamics damping="0.1" friction="0.2"/>
+    <dynamics damping="0.03" friction="0.2"/>
     <limit
       lower="-1.66"
@@ -306,5 +306,5 @@
     <axis
       xyz="0 1 0" />
-    <dynamics damping="0.1" friction="0.2"/>
+    <dynamics damping="0.03" friction="0.2"/>
     <limit
       lower="-1.75"
@@ -359,5 +359,5 @@
     <axis
       xyz="0 1 0" />
-    <dynamics damping="0.1" friction="0.2"/>
+    <dynamics damping="0.03" friction="0.2"/>
     <limit
       lower="0.56"
@@ -412,5 +412,5 @@
     <axis
       xyz="0 1 0" />
-    <dynamics damping="0.1" friction="0.2"/>
+    <dynamics damping="0.03" friction="0.2"/>
     <limit
       lower="-1.08"
@@ -465,5 +465,5 @@
     <axis
       xyz="1 0 0" />
-    <dynamics damping="0.1" friction="0.2"/>
+    <dynamics damping="0.03" friction="0.2"/>
     <limit
       lower="-1.05"
@@ -519,5 +519,5 @@
     <axis
       xyz="0 0 1" />
-    <dynamics damping="0.1" friction="0.2"/>
+    <dynamics damping="0.03" friction="0.2"/>
     <limit
       lower="-1.66"
@@ -573,5 +573,5 @@
     <axis
       xyz="0 1 0" />
-    <dynamics damping="0.1" friction="0.2"/>
+    <dynamics damping="0.03" friction="0.2"/>
     <limit
       lower="-1.75"
@@ -626,5 +626,5 @@
     <axis
       xyz="0 1 0" />
-    <dynamics damping="0.1" friction="0.2"/>
+    <dynamics damping="0.03" friction="0.2"/>
     <limit
       lower="0.56"
@@ -679,5 +679,5 @@
     <axis
       xyz="0 1 0" />
-    <dynamics damping="0.1" friction="0.2"/>
+    <dynamics damping="0.03" friction="0.2"/>
     <limit
       lower="-1.08"

File: src/robots/gr1t1_description/xacro/gazebo.xacro (robot description, xacro)
@@ -1,11 +1,12 @@
 <?xml version="1.0"?>
 <robot>
+  <!-- ros_control plugin -->
   <gazebo>
     <plugin filename="libgazebo_ros_control.so" name="gazebo_ros_control">
-      <robotNamespace>/gh1_gazebo</robotNamespace>
+      <robotNamespace>/gr1t1_gazebo</robotNamespace>
       <robotSimType>gazebo_ros_control/DefaultRobotHWSim</robotSimType>
     </plugin>
   </gazebo>
-  <!-- Show the trajectory of base_link center. -->
+  <!-- Show the trajectory of body center. -->
   <!-- <gazebo>
         <plugin name="3dplot" filename="libLinkPlot3DPlugin.so">
@@ -61,6 +62,6 @@
     <mu1>0.2</mu1>
     <mu2>0.2</mu2>
-    <kp value="1000000.0" />
-    <kd value="1.0" />
+    <kp value="1000000.0"/>
+    <kd value="1.0"/>
   </gazebo>
   <gazebo reference="imu_link">
@@ -98,6 +99,6 @@
     <mu2>1.0</mu2>
     <self_collide>1</self_collide>
-    <kp value="1000000.0" />
-    <kd value="1.0" />
+    <kp value="1000000.0"/>
+    <kd value="1.0"/>
     <material>Gazebo/DarkGrey</material>
   </gazebo>
@@ -106,6 +107,6 @@
     <mu2>1.0</mu2>
     <self_collide>1</self_collide>
-    <kp value="1000000.0" />
-    <kd value="1.0" />
+    <kp value="1000000.0"/>
+    <kd value="1.0"/>
     <material>Gazebo/DarkGrey</material>
   </gazebo>
@@ -139,6 +140,6 @@
     <mu2>1.0</mu2>
     <self_collide>1</self_collide>
-    <kp value="1000000.0" />
-    <kd value="1.0" />
+    <kp value="1000000.0"/>
+    <kd value="1.0"/>
     <material>Gazebo/DarkGrey</material>
   </gazebo>
@@ -147,6 +148,6 @@
     <mu2>1.0</mu2>
     <self_collide>1</self_collide>
-    <kp value="1000000.0" />
-    <kd value="1.0" />
+    <kp value="1000000.0"/>
+    <kd value="1.0"/>
     <material>Gazebo/DarkGrey</material>
   </gazebo>

Commit message: 机身质量有问题,修改为正确数值

File: src/robots/gh1_description/xacro/robot.xacro (robot description, xacro)
@@ -61,12 +61,12 @@
         rpy="0 0 0" />
       <mass
-        value="10.935" />
-      <inertia
-        ixx="0.12979"
-        ixy="1.4382E-06"
-        ixz="-0.00016277"
-        iyy="0.099343"
-        iyz="-2.2433E-07"
-        izz="0.067516" />
+        value="23.55" />
+      <inertia
+        ixx="0.46786000"
+        ixy="0"
+        ixz="0"
+        iyy="0.37758500"
+        iyz="0"
+        izz="0.21744500" />
     </inertial>
     <visual>

Commit message: 配合qr_wl控制软件20241030晚提交的版本，成功控制人形AI运动。

File: src/robots/gh1_description/xacro/robot.xacro (robot description, xacro)
@@ -37,5 +37,5 @@
     <link name="world" />
     <joint name="base_static_joint" type="fixed">
-      <origin rpy="0 0 0" xyz="0 0 -0.5" />
+      <origin rpy="0 0 0" xyz="0 0 1.2" />
       <parent link="world" />
       <child link="base" />
@@ -58,5 +58,5 @@
     <inertial>
       <origin
-        xyz="-0.0057915 -8.0007E-06 -0.045258"
+        xyz="-0.0057915 -8.0007E-06 0.16"
         rpy="0 0 0" />
       <mass
@@ -197,5 +197,4 @@
     <axis
       xyz="1 0 0" />
-    <dynamics damping="0.03" friction="0.2"/>
     <limit
       lower="-0.17"
@@ -253,8 +252,7 @@
     <axis
       xyz="0 0 1" />
-    <dynamics damping="0.03" friction="0.2"/>
-    <limit
-      lower="-1.66"
-      upper="1.66"
+    <limit
+      lower="-0.1"
+      upper="0.1"
       effort="70"
       velocity="12.552" />
@@ -306,5 +304,4 @@
     <axis
       xyz="0 1 0" />
-    <dynamics damping="0.03" friction="0.2"/>
     <limit
       lower="-1.75"
@@ -359,7 +356,6 @@
     <axis
       xyz="0 1 0" />
-    <dynamics damping="0.03" friction="0.2"/>
-    <limit
-      lower="0.56"
+    <limit
+      lower="0"
       upper="2.23"
       effort="120"
@@ -395,5 +391,5 @@
       </material>
     </visual>
-    <collision>
+    <!-- <collision>
       <origin
         xyz="0.025 0 -0.045"
@@ -401,4 +397,28 @@
       <geometry>
         <box size="0.25 0.05 0.02"/>
+      </geometry>
+    </collision> -->
+    <collision>
+      <origin
+        xyz="0.02 0 -0.04"
+        rpy="0 1.57 0" />
+      <geometry>
+        <cylinder radius="0.015" length="0.22"/>
+      </geometry>
+    </collision>
+    <collision>
+      <origin
+        xyz="0.13 0 -0.04"
+        rpy="0 0 0" />
+      <geometry>
+        <sphere radius="0.015"/>
+      </geometry>
+    </collision>
+    <collision>
+      <origin
+        xyz="-0.09 0 -0.04"
+        rpy="0 0 0" />
+      <geometry>
+        <sphere radius="0.015"/>
       </geometry>
     </collision>
@@ -412,5 +432,4 @@
     <axis
       xyz="0 1 0" />
-    <dynamics damping="0.03" friction="0.2"/>
     <limit
       lower="-1.08"
@@ -465,5 +484,4 @@
     <axis
       xyz="1 0 0" />
-    <dynamics damping="0.03" friction="0.2"/>
     <limit
       lower="-1.05"
@@ -519,8 +537,7 @@
     <axis
       xyz="0 0 1" />
-    <dynamics damping="0.03" friction="0.2"/>
-    <limit
-      lower="-1.66"
-      upper="1.66"
+    <limit
+      lower="-0.1"
+      upper="0.1"
       effort="70"
       velocity="12.552" />
@@ -573,5 +590,4 @@
     <axis
       xyz="0 1 0" />
-    <dynamics damping="0.03" friction="0.2"/>
     <limit
       lower="-1.75"
@@ -626,7 +642,6 @@
     <axis
       xyz="0 1 0" />
-    <dynamics damping="0.03" friction="0.2"/>
-    <limit
-      lower="0.56"
+    <limit
+      lower="0"
       upper="2.23"
       effort="120"
@@ -662,5 +677,5 @@
       </material>
     </visual>
-    <collision>
+    <!-- <collision>
       <origin
         xyz="0.025 0 -0.045"
@@ -668,4 +683,28 @@
       <geometry>
         <box size="0.25 0.05 0.02"/>
+      </geometry>
+    </collision> -->
+    <collision>
+      <origin
+        xyz="0.02 0 -0.04"
+        rpy="0 1.57 0" />
+      <geometry>
+        <cylinder radius="0.015" length="0.22"/>
+      </geometry>
+    </collision>
+    <collision>
+      <origin
+        xyz="0.13 0 -0.04"
+        rpy="0 0 0" />
+      <geometry>
+        <sphere radius="0.015"/>
+      </geometry>
+    </collision>
+    <collision>
+      <origin
+        xyz="-0.09 0 -0.04"
+        rpy="0 0 0" />
+      <geometry>
+        <sphere radius="0.015"/>
       </geometry>
     </collision>
@@ -679,5 +718,4 @@
     <axis
       xyz="0 1 0" />
-    <dynamics damping="0.03" friction="0.2"/>
     <limit
       lower="-1.08"

Commit message: 修改人形的debug默认位置与初始关节角

File: src/robots/gh1_description/xacro/robot.xacro (robot description, xacro)
@@ -37,5 +37,5 @@
     <link name="world" />
     <joint name="base_static_joint" type="fixed">
-      <origin rpy="0 0 0" xyz="0 0 1.2" />
+      <origin rpy="0 0 0" xyz="0 0 0.0" />
       <parent link="world" />
       <child link="base" />
