Commit message: 初步成功启动了关节控制器,hardware接口直接使用gazebo的就可以了,将urdf依赖添加到cmakelist中不然才创建不了urdf model对象接收description,实现不了接收参数文件中的joint名称来动态声明关节控制器名字

File: src/robot_description/gh1/xacro/robot.xacro (robot description, xacro)
@@ -76,5 +76,5 @@
       <geometry>
         <mesh
-          filename="/home/ww/Documents/simulation_all_ros2/src/robot_description/gh1/meshes/base_link.STL" />
+          filename="/home/wl/Documents/simulation_all_ros2/src/robot_description/gh1/meshes/base_link.STL" />
       </geometry>
       <material
@@ -168,5 +168,5 @@
       <geometry>
         <mesh
-          filename="/home/ww/Documents/simulation_all_ros2/src/robot_description/gh1/meshes/L1_link.STL" />
+          filename="/home/wl/Documents/simulation_all_ros2/src/robot_description/gh1/meshes/L1_link.STL" />
       </geometry>
       <material
@@ -225,5 +225,5 @@
       <geometry>
         <mesh
-          filename="/home/ww/Documents/simulation_all_ros2/src/robot_description/gh1/meshes/L2_link.STL" />
+          filename="/home/wl/Documents/simulation_all_ros2/src/robot_description/gh1/meshes/L2_link.STL" />
       </geometry>
       <material
@@ -279,5 +279,5 @@
       <geometry>
         <mesh
-          filename="/home/ww/Documents/simulation_all_ros2/src/robot_description/gh1/meshes/L3_link.STL" />
+          filename="/home/wl/Documents/simulation_all_ros2/src/robot_description/gh1/meshes/L3_link.STL" />
       </geometry>
       <material
@@ -331,5 +331,5 @@
       <geometry>
         <mesh
-          filename="/home/ww/Documents/simulation_all_ros2/src/robot_description/gh1/meshes/L4_link.STL" />
+          filename="/home/wl/Documents/simulation_all_ros2/src/robot_description/gh1/meshes/L4_link.STL" />
       </geometry>
       <material
@@ -383,5 +383,5 @@
       <geometry>
         <mesh
-          filename="/home/ww/Documents/simulation_all_ros2/src/robot_description/gh1/meshes/L5_link.STL" />
+          filename="/home/wl/Documents/simulation_all_ros2/src/robot_description/gh1/meshes/L5_link.STL" />
       </geometry>
       <material
@@ -459,5 +459,5 @@
       <geometry>
         <mesh
-          filename="/home/ww/Documents/simulation_all_ros2/src/robot_description/gh1/meshes/R1_link.STL" />
+          filename="/home/wl/Documents/simulation_all_ros2/src/robot_description/gh1/meshes/R1_link.STL" />
       </geometry>
       <material
@@ -512,5 +512,5 @@
       <geometry>
         <mesh
-          filename="/home/ww/Documents/simulation_all_ros2/src/robot_description/gh1/meshes/R2_link.STL" />
+          filename="/home/wl/Documents/simulation_all_ros2/src/robot_description/gh1/meshes/R2_link.STL" />
       </geometry>
       <material
@@ -565,5 +565,5 @@
       <geometry>
         <mesh
-          filename="/home/ww/Documents/simulation_all_ros2/src/robot_description/gh1/meshes/R3_link.STL" />
+          filename="/home/wl/Documents/simulation_all_ros2/src/robot_description/gh1/meshes/R3_link.STL" />
       </geometry>
       <material
@@ -617,5 +617,5 @@
       <geometry>
         <mesh
-          filename="/home/ww/Documents/simulation_all_ros2/src/robot_description/gh1/meshes/R4_link.STL" />
+          filename="/home/wl/Documents/simulation_all_ros2/src/robot_description/gh1/meshes/R4_link.STL" />
       </geometry>
       <material
@@ -669,5 +669,5 @@
       <geometry>
         <mesh
-          filename="/home/ww/Documents/simulation_all_ros2/src/robot_description/gh1/meshes/R5_link.STL" />
+          filename="/home/wl/Documents/simulation_all_ros2/src/robot_description/gh1/meshes/R5_link.STL" />
       </geometry>
       <material
@@ -724,103 +724,15 @@
       velocity="46.024" />
   </joint>
-  <transmission name="l_hip_roll_tran">
-    <type>transmission_interface/SimpleTransmission</type>
+  <ros2_control name="gh1_gazebo" type="system">
+    <hardware>
+      <plugin>fake_components/GenericSystem</plugin>
+    </hardware>
     <joint name="l_hip_roll">
-      <hardwareInterface>hardware_interface/EffortJointInterface</hardwareInterface>
+      <command_interface name="effort">
+      </command_interface>
+      <state_interface name="position"/>
+      <state_interface name="velocity"/>
+      <state_interface name="effort"/>
     </joint>
-    <actuator name="l_hip_roll_motor">
-      <hardwareInterface>hardware_interface/EffortJointInterface</hardwareInterface>
-      <mechanicalReduction>&quot;1&quot;</mechanicalReduction>
-    </actuator>
-  </transmission>
-  <transmission name="l_hip_yaw_tran">
-    <type>transmission_interface/SimpleTransmission</type>
-    <joint name="l_hip_yaw">
-      <hardwareInterface>hardware_interface/EffortJointInterface</hardwareInterface>
-    </joint>
-    <actuator name="l_hip_yaw_motor">
-      <hardwareInterface>hardware_interface/EffortJointInterface</hardwareInterface>
-      <mechanicalReduction>&quot;1&quot;</mechanicalReduction>
-    </actuator>
-  </transmission>
-  <transmission name="l_hip_pitch_tran">
-    <type>transmission_interface/SimpleTransmission</type>
-    <joint name="l_hip_pitch">
-      <hardwareInterface>hardware_interface/EffortJointInterface</hardwareInterface>
-    </joint>
-    <actuator name="l_hip_pitch_motor">
-      <hardwareInterface>hardware_interface/EffortJointInterface</hardwareInterface>
-      <mechanicalReduction>&quot;1&quot;</mechanicalReduction>
-    </actuator>
-  </transmission>
-  <transmission name="l_knee_pitch_tran">
-    <type>transmission_interface/SimpleTransmission</type>
-    <joint name="l_knee_pitch">
-      <hardwareInterface>hardware_interface/EffortJointInterface</hardwareInterface>
-    </joint>
-    <actuator name="l_knee_pitch_motor">
-      <hardwareInterface>hardware_interface/EffortJointInterface</hardwareInterface>
-      <mechanicalReduction>&quot;1&quot;</mechanicalReduction>
-    </actuator>
-  </transmission>
-  <transmission name="l_ankle_pitch_tran">
-    <type>transmission_interface/SimpleTransmission</type>
-    <joint name="l_ankle_pitch">
-      <hardwareInterface>hardware_interface/EffortJointInterface</hardwareInterface>
-    </joint>
-    <actuator name="l_ankle_pitch_motor">
-      <hardwareInterface>hardware_interface/EffortJointInterface</hardwareInterface>
-      <mechanicalReduction>&quot;1&quot;</mechanicalReduction>
-    </actuator>
-  </transmission>
-  <transmission name="r_hip_roll_tran">
-    <type>transmission_interface/SimpleTransmission</type>
-    <joint name="r_hip_roll">
-      <hardwareInterface>hardware_interface/EffortJointInterface</hardwareInterface>
-    </joint>
-    <actuator name="r_hip_roll_motor">
-      <hardwareInterface>hardware_interface/EffortJointInterface</hardwareInterface>
-      <mechanicalReduction>&quot;1&quot;</mechanicalReduction>
-    </actuator>
-  </transmission>
-  <transmission name="r_hip_yaw_tran">
-    <type>transmission_interface/SimpleTransmission</type>
-    <joint name="r_hip_yaw">
-      <hardwareInterface>hardware_interface/EffortJointInterface</hardwareInterface>
-    </joint>
-    <actuator name="r_hip_yaw_motor">
-      <hardwareInterface>hardware_interface/EffortJointInterface</hardwareInterface>
-      <mechanicalReduction>&quot;1&quot;</mechanicalReduction>
-    </actuator>
-  </transmission>
-  <transmission name="r_hip_pitch_tran">
-    <type>transmission_interface/SimpleTransmission</type>
-    <joint name="r_hip_pitch">
-      <hardwareInterface>hardware_interface/EffortJointInterface</hardwareInterface>
-    </joint>
-    <actuator name="r_hip_pitch_motor">
-      <hardwareInterface>hardware_interface/EffortJointInterface</hardwareInterface>
-      <mechanicalReduction>&quot;1&quot;</mechanicalReduction>
-    </actuator>
-  </transmission>
-  <transmission name="r_knee_pitch_tran">
-    <type>transmission_interface/SimpleTransmission</type>
-    <joint name="r_knee_pitch">
-      <hardwareInterface>hardware_interface/EffortJointInterface</hardwareInterface>
-    </joint>
-    <actuator name="r_knee_pitch_motor">
-      <hardwareInterface>hardware_interface/EffortJointInterface</hardwareInterface>
-      <mechanicalReduction>&quot;1&quot;</mechanicalReduction>
-    </actuator>
-  </transmission>
-  <transmission name="r_ankle_pitch_tran">
-    <type>transmission_interface/SimpleTransmission</type>
-    <joint name="r_ankle_pitch">
-      <hardwareInterface>hardware_interface/EffortJointInterface</hardwareInterface>
-    </joint>
-    <actuator name="r_ankle_pitch_motor">
-      <hardwareInterface>hardware_interface/EffortJointInterface</hardwareInterface>
-      <mechanicalReduction>&quot;1&quot;</mechanicalReduction>
-    </actuator>
-  </transmission>
+  </ros2_control>
 </robot>
