Commit message: .第一次实现了加载人形机器人模型

File: src/robot_description/gh1/xacro/gazebo.xacro (robot description, xacro)
@@ -7,26 +7,4 @@
     </plugin>
   </gazebo>
-  <!-- Show the trajectory of base_link center. -->
-  <!-- <gazebo>
-        <plugin name="3dplot" filename="libLinkPlot3DPlugin.so">
-            <frequency>10</frequency>
-            <plot>
-                <link>base</link>
-                <pose>0 0 0 0 0 0</pose>
-                <material>Gazebo/Yellow</material>
-            </plot>
-        </plugin>
-    </gazebo> -->
-  <!-- Show the trajectory of foot. You can add another trajectory about another foot. -->
-  <!-- <gazebo>
-        <plugin name="3dplot" filename="libLinkPlot3DPlugin.so">
-            <frequency>100</frequency>
-            <plot>
-                <link>FL_foot</link>
-                <pose>0 0 0 0 0 0</pose>
-                <material>Gazebo/Green</material>
-            </plot>
-        </plugin>
-    </gazebo> -->
   <gazebo>
     <plugin filename="libgazebo_ros_force.so" name="gazebo_ros_force">

File: src/robot_description/gh1/xacro/robot.xacro (robot description, xacro)
@@ -200,4 +200,5 @@
       lower="-0.17"
       upper="1.05"
+      value="1.00"
       effort="120"
       velocity="20.92" />

Commit message: 机器人的xacro文件中添加了ros2_control标签用于控制器启动识别,在gazebo_ros_force插件使用link_name替代bodyName

File: src/robot_description/gh1/xacro/gazebo.xacro (robot description, xacro)
@@ -3,5 +3,5 @@
   <gazebo>
     <plugin filename="libgazebo_ros_control.so" name="gazebo_ros_control">
-      <robotNamespace>/gh1_gazebo</robotNamespace>
+      <robotNamespace>gh1</robotNamespace>
       <robotSimType>gazebo_ros_control/DefaultRobotHWSim</robotSimType>
     </plugin>
@@ -9,6 +9,7 @@
   <gazebo>
     <plugin filename="libgazebo_ros_force.so" name="gazebo_ros_force">
-      <bodyName>body</bodyName>
+      <link_name>body</link_name>
       <topicName>/apply_force/body</topicName>
+      <force_frame>body</force_frame>
     </plugin>
   </gazebo>

File: src/robot_description/gh1/xacro/robot.xacro (robot description, xacro)
@@ -200,5 +200,4 @@
       lower="-0.17"
       upper="1.05"
-      value="1.00"
       effort="120"
       velocity="20.92" />
@@ -732,5 +731,5 @@
     <actuator name="l_hip_roll_motor">
       <hardwareInterface>hardware_interface/EffortJointInterface</hardwareInterface>
-      <mechanicalReduction>&quot;1&quot;</mechanicalReduction>
+      <mechanicalReduction>1</mechanicalReduction>
     </actuator>
   </transmission>
@@ -742,5 +741,5 @@
     <actuator name="l_hip_yaw_motor">
       <hardwareInterface>hardware_interface/EffortJointInterface</hardwareInterface>
-      <mechanicalReduction>&quot;1&quot;</mechanicalReduction>
+      <mechanicalReduction>1</mechanicalReduction>
     </actuator>
   </transmission>
@@ -752,5 +751,5 @@
     <actuator name="l_hip_pitch_motor">
       <hardwareInterface>hardware_interface/EffortJointInterface</hardwareInterface>
-      <mechanicalReduction>&quot;1&quot;</mechanicalReduction>
+      <mechanicalReduction>1</mechanicalReduction>
     </actuator>
   </transmission>
@@ -762,5 +761,5 @@
     <actuator name="l_knee_pitch_motor">
       <hardwareInterface>hardware_interface/EffortJointInterface</hardwareInterface>
-      <mechanicalReduction>&quot;1&quot;</mechanicalReduction>
+      <mechanicalReduction>1</mechanicalReduction>
     </actuator>
   </transmission>
@@ -772,5 +771,5 @@
     <actuator name="l_ankle_pitch_motor">
       <hardwareInterface>hardware_interface/EffortJointInterface</hardwareInterface>
-      <mechanicalReduction>&quot;1&quot;</mechanicalReduction>
+      <mechanicalReduction>1</mechanicalReduction>
     </actuator>
   </transmission>
@@ -782,5 +781,5 @@
     <actuator name="r_hip_roll_motor">
       <hardwareInterface>hardware_interface/EffortJointInterface</hardwareInterface>
-      <mechanicalReduction>&quot;1&quot;</mechanicalReduction>
+      <mechanicalReduction>1</mechanicalReduction>
     </actuator>
   </transmission>
@@ -792,5 +791,5 @@
     <actuator name="r_hip_yaw_motor">
       <hardwareInterface>hardware_interface/EffortJointInterface</hardwareInterface>
-      <mechanicalReduction>&quot;1&quot;</mechanicalReduction>
+      <mechanicalReduction>1</mechanicalReduction>
     </actuator>
   </transmission>
@@ -802,5 +801,5 @@
     <actuator name="r_hip_pitch_motor">
       <hardwareInterface>hardware_interface/EffortJointInterface</hardwareInterface>
-      <mechanicalReduction>&quot;1&quot;</mechanicalReduction>
+      <mechanicalReduction>1</mechanicalReduction>
     </actuator>
   </transmission>
@@ -812,5 +811,5 @@
     <actuator name="r_knee_pitch_motor">
       <hardwareInterface>hardware_interface/EffortJointInterface</hardwareInterface>
-      <mechanicalReduction>&quot;1&quot;</mechanicalReduction>
+      <mechanicalReduction>1</mechanicalReduction>
     </actuator>
   </transmission>
@@ -822,6 +821,73 @@
     <actuator name="r_ankle_pitch_motor">
       <hardwareInterface>hardware_interface/EffortJointInterface</hardwareInterface>
-      <mechanicalReduction>&quot;1&quot;</mechanicalReduction>
-    </actuator>
-  </transmission>
+      <mechanicalReduction>1</mechanicalReduction>
+    </actuator>
+  </transmission>
+  <ros2_control name="gh1" type="loan_command">
+    <hardware>
+      <plugin>robot_joint_controller/RobotJointController</plugin>
+      <param name="example_param_hw_start_duration_sec">2.0</param>
+      <param name="example_param_hw_stop_duration_sec">3.0</param>
+    </hardware>
+    <joint name="l_hip_roll">
+      <command_interface name="effort"/>
+      <state_interface name="position"/>
+      <state_interface name="velocity"/>
+      <state_interface name="effort"/>
+    </joint>
+    <joint name="l_hip_yaw">
+      <command_interface name="effort"/>
+      <state_interface name="position"/>
+      <state_interface name="velocity"/>
+      <state_interface name="effort"/>
+    </joint>
+    <joint name="l_hip_pitch">
+      <command_interface name="effort"/>
+      <state_interface name="position"/>
+      <state_interface name="velocity"/>
+      <state_interface name="effort"/>
+    </joint>
+    <joint name="l_knee_pitch">
+      <command_interface name="effort"/>
+      <state_interface name="position"/>
+      <state_interface name="velocity"/>
+      <state_interface name="effort"/>
+    </joint>
+    <joint name="l_ankle_pitch">
+      <command_interface name="effort"/>
+      <state_interface name="position"/>
+      <state_interface name="velocity"/>
+      <state_interface name="effort"/>
+    </joint>
+    <joint name="r_hip_roll">
+      <command_interface name="effort"/>
+      <state_interface name="position"/>
+      <state_interface name="velocity"/>
+      <state_interface name="effort"/>
+    </joint>
+    <joint name="r_hip_yaw">
+      <command_interface name="effort"/>
+      <state_interface name="position"/>
+      <state_interface name="velocity"/>
+      <state_interface name="effort"/>
+    </joint>
+    <joint name="r_hip_pitch">
+      <command_interface name="effort"/>
+      <state_interface name="position"/>
+      <state_interface name="velocity"/>
+      <state_interface name="effort"/>
+    </joint>
+    <joint name="r_knee_pitch">
+      <command_interface name="effort"/>
+      <state_interface name="position"/>
+      <state_interface name="velocity"/>
+      <state_interface name="effort"/>
+    </joint>
+    <joint name="r_ankle_pitch">
+      <command_interface name="effort"/>
+      <state_interface name="position"/>
+      <state_interface name="velocity"/>
+      <state_interface name="effort"/>
+    </joint>
+  </ros2_control>
 </robot>

Commit message: .将除了l_hip_roll以及l_thigh_roll以外的注释,先针对一个关节进行修改

File: src/robot_description/gh1/xacro/gazebo.xacro (robot description, xacro)
@@ -55,5 +55,5 @@
     <material>Gazebo/DarkGrey</material>
   </gazebo>
-  <gazebo reference="l_thigh_yaw">
+<!-- <gazebo reference="l_thigh_yaw">
     <mu1>0.2</mu1>
     <mu2>0.2</mu2>
@@ -129,4 +129,4 @@
     <kd value="1.0" />
     <material>Gazebo/DarkGrey</material>
-  </gazebo>
+  </gazebo> -->
 </robot>

File: src/robot_description/gh1/xacro/robot.xacro (robot description, xacro)
@@ -130,15 +130,4 @@
     </collision>
   </link>
-  <link name="imu_link">
-    <visual>
-      <origin xyz="-0.0 0 -0.0" rpy="0 0 0" />
-      <geometry>
-        <box size="0.05 0.05 0.02" />
-      </geometry>
-      <material name="">
-        <color rgba="0.75294 0.75294 0.75294 1" />
-      </material>
-    </visual>
-  </link>
   <joint name="z_joint_imu" type="fixed">
     <origin xyz="-0.0 0 -0.0" rpy="0 0 0" />
@@ -146,42 +135,14 @@
     <child link="imu_link" />
   </joint>
-  <link
-    name="l_thigh_roll">
-    <inertial>
-      <origin
-        xyz="0.078159 0.0 0.003801"
-        rpy="0 0 0" />
-      <mass
-        value="2.19" />
-      <inertia
-        ixx="0.00262800"
-        ixy="0"
-        ixz="0"
-        iyy="0.00262800"
-        iyz="0"
-        izz="0.00394200" />
-    </inertial>
-    <visual>
-      <origin
-        xyz="0 0 0"
-        rpy="0 0 0" />
-      <geometry>
-        <mesh
-          filename="package://gh1/meshes/L1_link.STL" />
-      </geometry>
-      <material
-        name="">
-        <color
-          rgba="1 1 1 0.3" />
-      </material>
-    </visual>
-    <collision>
-      <origin
-        xyz="0.085 0 0"
-        rpy="0 0 0" />
-      <geometry>
-        <cylinder radius="0.06" length="0.06" />
-      </geometry>
-    </collision>
+  <link name="imu_link">
+    <visual>
+      <origin xyz="-0.0 0 -0.0" rpy="0 0 0" />
+      <geometry>
+        <box size="0.05 0.05 0.02" />
+      </geometry>
+      <material name="">
+        <color rgba="0.75294 0.75294 0.75294 1" />
+      </material>
+    </visual>
   </link>
   <joint
@@ -204,4 +165,43 @@
   </joint>
   <link
+    name="l_thigh_roll">
+    <inertial>
+      <origin
+        xyz="0.078159 0.0 0.003801"
+        rpy="0 0 0" />
+      <mass
+        value="2.19" />
+      <inertia
+        ixx="0.00262800"
+        ixy="0"
+        ixz="0"
+        iyy="0.00262800"
+        iyz="0"
+        izz="0.00394200" />
+    </inertial>
+    <visual>
+      <origin
+        xyz="0 0 0"
+        rpy="0 0 0" />
+      <geometry>
+        <mesh
+          filename="package://gh1/meshes/L1_link.STL" />
+      </geometry>
+      <material
+        name="">
+        <color
+          rgba="1 1 1 0.3" />
+      </material>
+    </visual>
+    <collision>
+      <origin
+        xyz="0.085 0 0"
+        rpy="0 0 0" />
+      <geometry>
+        <cylinder radius="0.06" length="0.06" />
+      </geometry>
+    </collision>
+  </link>
+  <!-- <link
     name="l_thigh_yaw">
     <inertial>
@@ -391,12 +391,4 @@
       </material>
     </visual>
-    <!-- <collision>
-      <origin
-        xyz="0.025 0 -0.045"
-        rpy="0 0 0" />
-      <geometry>
-        <box size="0.25 0.05 0.02"/>
-      </geometry>
-    </collision> -->
     <collision>
       <origin
@@ -677,12 +669,4 @@
       </material>
     </visual>
-    <!-- <collision>
-      <origin
-        xyz="0.025 0 -0.045"
-        rpy="0 0 0" />
-      <geometry>
-        <box size="0.25 0.05 0.02"/>
-      </geometry>
-    </collision> -->
     <collision>
       <origin
@@ -723,5 +707,5 @@
       effort="22"
       velocity="46.024" />
-  </joint>
+  </joint> -->
   <transmission name="l_hip_roll_tran">
     <type>transmission_interface/SimpleTransmission</type>
@@ -734,5 +718,5 @@
     </actuator>
   </transmission>
-  <transmission name="l_hip_yaw_tran">
+  <!-- <transmission name="l_hip_yaw_tran">
     <type>transmission_interface/SimpleTransmission</type>
     <joint name="l_hip_yaw">
@@ -823,6 +807,6 @@
       <mechanicalReduction>1</mechanicalReduction>
     </actuator>
-  </transmission>
-  <ros2_control name="gh1" type="loan_command">
+  </transmission> -->
+  <!-- <ros2_control name="gh1" type="loan_command">
     <hardware>
       <plugin>robot_joint_controller/RobotJointController</plugin>
@@ -890,4 +874,4 @@
       <state_interface name="effort"/>
     </joint>
-  </ros2_control>
+  </ros2_control> -->
 </robot>
