Commit message: .发现加载不出来模型的原因好像是由于stl模型文件不能正确的读取,同时gazebo_ros_force插件好像不能识别body link

File: src/robot_description/gh1/xacro/gazebo.xacro (robot description, xacro)
@@ -9,7 +9,6 @@
   <gazebo>
     <plugin filename="libgazebo_ros_force.so" name="gazebo_ros_force">
-      <link_name>body</link_name>
+      <link_name>base</link_name>
       <topicName>/apply_force/body</topicName>
-      <force_frame>body</force_frame>
     </plugin>
   </gazebo>
@@ -55,78 +54,3 @@
     <material>Gazebo/DarkGrey</material>
   </gazebo>
-<!-- <gazebo reference="l_thigh_yaw">
-    <mu1>0.2</mu1>
-    <mu2>0.2</mu2>
-    <self_collide>1</self_collide>
-    <material>Gazebo/DarkGrey</material>
-  </gazebo>
-  <gazebo reference="l_thigh_pitch">
-    <mu1>0.2</mu1>
-    <mu2>0.2</mu2>
-    <self_collide>1</self_collide>
-    <material>Gazebo/DarkGrey</material>
-  </gazebo>
-  <gazebo reference="l_shank_pitch">
-    <mu1>0.2</mu1>
-    <mu2>0.2</mu2>
-    <self_collide>1</self_collide>
-    <material>Gazebo/DarkGrey</material>
-  </gazebo>
-  <gazebo reference="l_foot_pitch">
-    <mu1>1.0</mu1>
-    <mu2>1.0</mu2>
-    <self_collide>1</self_collide>
-    <kp value="1000000.0" />
-    <kd value="1.0" />
-    <material>Gazebo/DarkGrey</material>
-  </gazebo>
-  <gazebo reference="l_foot_roll">
-    <mu1>1.0</mu1>
-    <mu2>1.0</mu2>
-    <self_collide>1</self_collide>
-    <kp value="1000000.0" />
-    <kd value="1.0" />
-    <material>Gazebo/DarkGrey</material>
-  </gazebo>
-  <!-- right leg -->
-  <gazebo reference="r_thigh_roll">
-    <mu1>0.2</mu1>
-    <mu2>0.2</mu2>
-    <self_collide>1</self_collide>
-    <material>Gazebo/DarkGrey</material>
-  </gazebo>
-  <gazebo reference="r_thigh_yaw">
-    <mu1>0.2</mu1>
-    <mu2>0.2</mu2>
-    <self_collide>1</self_collide>
-    <material>Gazebo/DarkGrey</material>
-  </gazebo>
-  <gazebo reference="r_thigh_pitch">
-    <mu1>0.2</mu1>
-    <mu2>0.2</mu2>
-    <self_collide>1</self_collide>
-    <material>Gazebo/DarkGrey</material>
-  </gazebo>
-  <gazebo reference="r_shank_pitch">
-    <mu1>0.2</mu1>
-    <mu2>0.2</mu2>
-    <self_collide>1</self_collide>
-    <material>Gazebo/DarkGrey</material>
-  </gazebo>
-  <gazebo reference="r_foot_pitch">
-    <mu1>1.0</mu1>
-    <mu2>1.0</mu2>
-    <self_collide>1</self_collide>
-    <kp value="1000000.0" />
-    <kd value="1.0" />
-    <material>Gazebo/DarkGrey</material>
-  </gazebo>
-  <gazebo reference="r_foot_roll">
-    <mu1>1.0</mu1>
-    <mu2>1.0</mu2>
-    <self_collide>1</self_collide>
-    <kp value="1000000.0" />
-    <kd value="1.0" />
-    <material>Gazebo/DarkGrey</material>
-  </gazebo> -->
 </robot>

File: src/robot_description/gh1/xacro/robot.xacro (robot description, xacro)
@@ -76,5 +76,5 @@
       <geometry>
         <mesh
-          filename="package://gh1/meshes/base_link.STL" />
+          filename="/home/wl/Documents/simulation_all_ros2/src/robot_description/gh1/meshes/base_link.STL" />
       </geometry>
       <material
@@ -129,4 +129,15 @@
       </geometry>
     </collision>
+  </link>
+  <link name="imu_link">
+    <visual>
+      <origin xyz="-0.0 0 -0.0" rpy="0 0 0" />
+      <geometry>
+        <box size="0.05 0.05 0.02" />
+      </geometry>
+      <material name="">
+        <color rgba="0.75294 0.75294 0.75294 1" />
+      </material>
+    </visual>
   </link>
   <joint name="z_joint_imu" type="fixed">
@@ -135,14 +146,42 @@
     <child link="imu_link" />
   </joint>
-  <link name="imu_link">
-    <visual>
-      <origin xyz="-0.0 0 -0.0" rpy="0 0 0" />
-      <geometry>
-        <box size="0.05 0.05 0.02" />
-      </geometry>
-      <material name="">
-        <color rgba="0.75294 0.75294 0.75294 1" />
-      </material>
-    </visual>
+  <link
+    name="l_thigh_roll">
+    <inertial>
+      <origin
+        xyz="0.078159 0.0 0.003801"
+        rpy="0 0 0" />
+      <mass
+        value="2.19" />
+      <inertia
+        ixx="0.00262800"
+        ixy="0"
+        ixz="0"
+        iyy="0.00262800"
+        iyz="0"
+        izz="0.00394200" />
+    </inertial>
+    <visual>
+      <origin
+        xyz="0 0 0"
+        rpy="0 0 0" />
+      <geometry>
+        <mesh
+          filename="/home/wl/Documents/simulation_all_ros2/src/robot_description/gh1/meshes/L1_link.STL" />
+      </geometry>
+      <material
+        name="">
+        <color
+          rgba="1 1 1 0.3" />
+      </material>
+    </visual>
+    <collision>
+      <origin
+        xyz="0.085 0 0"
+        rpy="0 0 0" />
+      <geometry>
+        <cylinder radius="0.06" length="0.06" />
+      </geometry>
+    </collision>
   </link>
   <joint
@@ -165,43 +204,4 @@
   </joint>
   <link
-    name="l_thigh_roll">
-    <inertial>
-      <origin
-        xyz="0.078159 0.0 0.003801"
-        rpy="0 0 0" />
-      <mass
-        value="2.19" />
-      <inertia
-        ixx="0.00262800"
-        ixy="0"
-        ixz="0"
-        iyy="0.00262800"
-        iyz="0"
-        izz="0.00394200" />
-    </inertial>
-    <visual>
-      <origin
-        xyz="0 0 0"
-        rpy="0 0 0" />
-      <geometry>
-        <mesh
-          filename="package://gh1/meshes/L1_link.STL" />
-      </geometry>
-      <material
-        name="">
-        <color
-          rgba="1 1 1 0.3" />
-      </material>
-    </visual>
-    <collision>
-      <origin
-        xyz="0.085 0 0"
-        rpy="0 0 0" />
-      <geometry>
-        <cylinder radius="0.06" length="0.06" />
-      </geometry>
-    </collision>
-  </link>
-  <!-- <link
     name="l_thigh_yaw">
     <inertial>
@@ -225,5 +225,5 @@
       <geometry>
         <mesh
-          filename="package://gh1/meshes/L2_link.STL" />
+          filename="/home/wl/Documents/simulation_all_ros2/src/robot_description/gh1/meshes/L2_link.STL" />
       </geometry>
       <material
@@ -279,5 +279,5 @@
       <geometry>
         <mesh
-          filename="package://gh1/meshes/L3_link.STL" />
+          filename="/home/wl/Documents/simulation_all_ros2/src/robot_description/gh1/meshes/L3_link.STL" />
       </geometry>
       <material
@@ -331,5 +331,5 @@
       <geometry>
         <mesh
-          filename="package://gh1/meshes/L4_link.STL" />
+          filename="/home/wl/Documents/simulation_all_ros2/src/robot_description/gh1/meshes/L4_link.STL" />
       </geometry>
       <material
@@ -383,12 +383,20 @@
       <geometry>
         <mesh
-          filename="package://gh1/meshes/L5_link.STL" />
-      </geometry>
-      <material
-        name="">
-        <color
-          rgba="1 1 1 0.3" />
-      </material>
-    </visual>
+          filename="/home/wl/Documents/simulation_all_ros2/src/robot_description/gh1/meshes/L5_link.STL" />
+      </geometry>
+      <material
+        name="">
+        <color
+          rgba="1 1 1 0.3" />
+      </material>
+    </visual>
+    <!-- <collision>
+      <origin
+        xyz="0.025 0 -0.045"
+        rpy="0 0 0" />
+      <geometry>
+        <box size="0.25 0.05 0.02"/>
+      </geometry>
+    </collision> -->
     <collision>
       <origin
@@ -451,5 +459,5 @@
       <geometry>
         <mesh
-          filename="package://gh1/meshes/R1_link.STL" />
+          filename="/home/wl/Documents/simulation_all_ros2/src/robot_description/gh1/meshes/R1_link.STL" />
       </geometry>
       <material
@@ -504,5 +512,5 @@
       <geometry>
         <mesh
-          filename="package://gh1/meshes/R2_link.STL" />
+          filename="/home/wl/Documents/simulation_all_ros2/src/robot_description/gh1/meshes/R2_link.STL" />
       </geometry>
       <material
@@ -557,5 +565,5 @@
       <geometry>
         <mesh
-          filename="package://gh1/meshes/R3_link.STL" />
+          filename="/home/wl/Documents/simulation_all_ros2/src/robot_description/gh1/meshes/R3_link.STL" />
       </geometry>
       <material
@@ -609,5 +617,5 @@
       <geometry>
         <mesh
-          filename="package://gh1/meshes/R4_link.STL" />
+          filename="/home/wl/Documents/simulation_all_ros2/src/robot_description/gh1/meshes/R4_link.STL" />
       </geometry>
       <material
@@ -661,12 +669,20 @@
       <geometry>
         <mesh
-          filename="package://gh1/meshes/R5_link.STL" />
-      </geometry>
-      <material
-        name="">
-        <color
-          rgba="1 1 1 0.3" />
-      </material>
-    </visual>
+          filename="/home/wl/Documents/simulation_all_ros2/src/robot_description/gh1/meshes/R5_link.STL" />
+      </geometry>
+      <material
+        name="">
+        <color
+          rgba="1 1 1 0.3" />
+      </material>
+    </visual>
+    <!-- <collision>
+      <origin
+        xyz="0.025 0 -0.045"
+        rpy="0 0 0" />
+      <geometry>
+        <box size="0.25 0.05 0.02"/>
+      </geometry>
+    </collision> -->
     <collision>
       <origin
@@ -707,5 +723,5 @@
       effort="22"
       velocity="46.024" />
-  </joint> -->
+  </joint>
   <transmission name="l_hip_roll_tran">
     <type>transmission_interface/SimpleTransmission</type>
@@ -715,8 +731,8 @@
     <actuator name="l_hip_roll_motor">
       <hardwareInterface>hardware_interface/EffortJointInterface</hardwareInterface>
-      <mechanicalReduction>1</mechanicalReduction>
-    </actuator>
-  </transmission>
-  <!-- <transmission name="l_hip_yaw_tran">
+      <mechanicalReduction>&quot;1&quot;</mechanicalReduction>
+    </actuator>
+  </transmission>
+  <transmission name="l_hip_yaw_tran">
     <type>transmission_interface/SimpleTransmission</type>
     <joint name="l_hip_yaw">
@@ -725,5 +741,5 @@
     <actuator name="l_hip_yaw_motor">
       <hardwareInterface>hardware_interface/EffortJointInterface</hardwareInterface>
-      <mechanicalReduction>1</mechanicalReduction>
+      <mechanicalReduction>&quot;1&quot;</mechanicalReduction>
     </actuator>
   </transmission>
@@ -735,5 +751,5 @@
     <actuator name="l_hip_pitch_motor">
       <hardwareInterface>hardware_interface/EffortJointInterface</hardwareInterface>
-      <mechanicalReduction>1</mechanicalReduction>
+      <mechanicalReduction>&quot;1&quot;</mechanicalReduction>
     </actuator>
   </transmission>
@@ -745,5 +761,5 @@
     <actuator name="l_knee_pitch_motor">
       <hardwareInterface>hardware_interface/EffortJointInterface</hardwareInterface>
-      <mechanicalReduction>1</mechanicalReduction>
+      <mechanicalReduction>&quot;1&quot;</mechanicalReduction>
     </actuator>
   </transmission>
@@ -755,5 +771,5 @@
     <actuator name="l_ankle_pitch_motor">
       <hardwareInterface>hardware_interface/EffortJointInterface</hardwareInterface>
-      <mechanicalReduction>1</mechanicalReduction>
+      <mechanicalReduction>&quot;1&quot;</mechanicalReduction>
     </actuator>
   </transmission>
@@ -765,5 +781,5 @@
     <actuator name="r_hip_roll_motor">
       <hardwareInterface>hardware_interface/EffortJointInterface</hardwareInterface>
-      <mechanicalReduction>1</mechanicalReduction>
+      <mechanicalReduction>&quot;1&quot;</mechanicalReduction>
     </actuator>
   </transmission>
@@ -775,5 +791,5 @@
     <actuator name="r_hip_yaw_motor">
       <hardwareInterface>hardware_interface/EffortJointInterface</hardwareInterface>
-      <mechanicalReduction>1</mechanicalReduction>
+      <mechanicalReduction>&quot;1&quot;</mechanicalReduction>
     </actuator>
   </transmission>
@@ -785,5 +801,5 @@
     <actuator name="r_hip_pitch_motor">
       <hardwareInterface>hardware_interface/EffortJointInterface</hardwareInterface>
-      <mechanicalReduction>1</mechanicalReduction>
+      <mechanicalReduction>&quot;1&quot;</mechanicalReduction>
     </actuator>
   </transmission>
@@ -795,5 +811,5 @@
     <actuator name="r_knee_pitch_motor">
       <hardwareInterface>hardware_interface/EffortJointInterface</hardwareInterface>
-      <mechanicalReduction>1</mechanicalReduction>
+      <mechanicalReduction>&quot;1&quot;</mechanicalReduction>
     </actuator>
   </transmission>
@@ -805,73 +821,6 @@
     <actuator name="r_ankle_pitch_motor">
       <hardwareInterface>hardware_interface/EffortJointInterface</hardwareInterface>
-      <mechanicalReduction>1</mechanicalReduction>
-    </actuator>
-  </transmission> -->
-  <!-- <ros2_control name="gh1" type="loan_command">
-    <hardware>
-      <plugin>robot_joint_controller/RobotJointController</plugin>
-      <param name="example_param_hw_start_duration_sec">2.0</param>
-      <param name="example_param_hw_stop_duration_sec">3.0</param>
-    </hardware>
-    <joint name="l_hip_roll">
-      <command_interface name="effort"/>
-      <state_interface name="position"/>
-      <state_interface name="velocity"/>
-      <state_interface name="effort"/>
-    </joint>
-    <joint name="l_hip_yaw">
-      <command_interface name="effort"/>
-      <state_interface name="position"/>
-      <state_interface name="velocity"/>
-      <state_interface name="effort"/>
-    </joint>
-    <joint name="l_hip_pitch">
-      <command_interface name="effort"/>
-      <state_interface name="position"/>
-      <state_interface name="velocity"/>
-      <state_interface name="effort"/>
-    </joint>
-    <joint name="l_knee_pitch">
-      <command_interface name="effort"/>
-      <state_interface name="position"/>
-      <state_interface name="velocity"/>
-      <state_interface name="effort"/>
-    </joint>
-    <joint name="l_ankle_pitch">
-      <command_interface name="effort"/>
-      <state_interface name="position"/>
-      <state_interface name="velocity"/>
-      <state_interface name="effort"/>
-    </joint>
-    <joint name="r_hip_roll">
-      <command_interface name="effort"/>
-      <state_interface name="position"/>
-      <state_interface name="velocity"/>
-      <state_interface name="effort"/>
-    </joint>
-    <joint name="r_hip_yaw">
-      <command_interface name="effort"/>
-      <state_interface name="position"/>
-      <state_interface name="velocity"/>
-      <state_interface name="effort"/>
-    </joint>
-    <joint name="r_hip_pitch">
-      <command_interface name="effort"/>
-      <state_interface name="position"/>
-      <state_interface name="velocity"/>
-      <state_interface name="effort"/>
-    </joint>
-    <joint name="r_knee_pitch">
-      <command_interface name="effort"/>
-      <state_interface name="position"/>
-      <state_interface name="velocity"/>
-      <state_interface name="effort"/>
-    </joint>
-    <joint name="r_ankle_pitch">
-      <command_interface name="effort"/>
-      <state_interface name="position"/>
-      <state_interface name="velocity"/>
-      <state_interface name="effort"/>
-    </joint>
-  </ros2_control> -->
+      <mechanicalReduction>&quot;1&quot;</mechanicalReduction>
+    </actuator>
+  </transmission>
 </robot>
