Commit message: .第一次完成的成功启动并配置了人形下肢的控制器以及对应gazebo_ros2_control接口

File: src/robot_description/gh1/xacro/gazebo.xacro (robot description, xacro)
@@ -59,3 +59,62 @@
     <material>Gazebo/DarkGrey</material>
   </gazebo>
+  <gazebo reference="l_thigh_yaw">
+    <mu1>0.2</mu1>
+    <mu2>0.2</mu2>
+    <self_collide>1</self_collide>
+    <material>Gazebo/DarkGrey</material>
+  </gazebo>
+  <gazebo reference="l_thigh_pitch">
+    <mu1>0.2</mu1>
+    <mu2>0.2</mu2>
+    <self_collide>1</self_collide>
+    <material>Gazebo/DarkGrey</material>
+  </gazebo>
+  <gazebo reference="l_shank_pitch">
+    <mu1>0.2</mu1>
+    <mu2>0.2</mu2>
+    <self_collide>1</self_collide>
+    <material>Gazebo/DarkGrey</material>
+  </gazebo>
+  <gazebo reference="l_foot_pitch">
+    <mu1>1.0</mu1>
+    <mu2>1.0</mu2>
+    <self_collide>1</self_collide>
+    <kp value="1000000.0" />
+    <kd value="1.0" />
+    <material>Gazebo/DarkGrey</material>
+  </gazebo>
+  <!-- right leg -->
+  <gazebo reference="r_thigh_roll">
+    <mu1>0.2</mu1>
+    <mu2>0.2</mu2>
+    <self_collide>1</self_collide>
+    <material>Gazebo/DarkGrey</material>
+  </gazebo>
+  <gazebo reference="r_thigh_yaw">
+    <mu1>0.2</mu1>
+    <mu2>0.2</mu2>
+    <self_collide>1</self_collide>
+    <material>Gazebo/DarkGrey</material>
+  </gazebo>
+  <gazebo reference="r_thigh_pitch">
+    <mu1>0.2</mu1>
+    <mu2>0.2</mu2>
+    <self_collide>1</self_collide>
+    <material>Gazebo/DarkGrey</material>
+  </gazebo>
+  <gazebo reference="r_shank_pitch">
+    <mu1>0.2</mu1>
+    <mu2>0.2</mu2>
+    <self_collide>1</self_collide>
+    <material>Gazebo/DarkGrey</material>
+  </gazebo>
+  <gazebo reference="r_foot_pitch">
+    <mu1>1.0</mu1>
+    <mu2>1.0</mu2>
+    <self_collide>1</self_collide>
+    <kp value="1000000.0" />
+    <kd value="1.0" />
+    <material>Gazebo/DarkGrey</material>
+  </gazebo>
 </robot>

File: src/robot_description/gh1/xacro/robot.xacro (robot description, xacro)
@@ -130,15 +130,4 @@
     </collision>
   </link>
-  <link name="imu_link">
-    <visual>
-      <origin xyz="-0.0 0 -0.0" rpy="0 0 0" />
-      <geometry>
-        <box size="0.05 0.05 0.02" />
-      </geometry>
-      <material name="">
-        <color rgba="0.75294 0.75294 0.75294 1" />
-      </material>
-    </visual>
-  </link>
   <joint name="z_joint_imu" type="fixed">
     <origin xyz="-0.0 0 -0.0" rpy="0 0 0" />
@@ -146,42 +135,14 @@
     <child link="imu_link" />
   </joint>
-  <link
-    name="l_thigh_roll">
-    <inertial>
-      <origin
-        xyz="0.078159 0.0 0.003801"
-        rpy="0 0 0" />
-      <mass
-        value="2.19" />
-      <inertia
-        ixx="0.00262800"
-        ixy="0"
-        ixz="0"
-        iyy="0.00262800"
-        iyz="0"
-        izz="0.00394200" />
-    </inertial>
-    <visual>
-      <origin
-        xyz="0 0 0"
-        rpy="0 0 0" />
-      <geometry>
-        <mesh
-          filename="/home/wl/Documents/simulation_all_ros2/src/robot_description/gh1/meshes/L1_link.STL" />
-      </geometry>
-      <material
-        name="">
-        <color
-          rgba="1 1 1 0.3" />
-      </material>
-    </visual>
-    <collision>
-      <origin
-        xyz="0.085 0 0"
-        rpy="0 0 0" />
-      <geometry>
-        <cylinder radius="0.06" length="0.06" />
-      </geometry>
-    </collision>
+  <link name="imu_link">
+    <visual>
+      <origin xyz="-0.0 0 -0.0" rpy="0 0 0" />
+      <geometry>
+        <box size="0.05 0.05 0.02" />
+      </geometry>
+      <material name="">
+        <color rgba="0.75294 0.75294 0.75294 1" />
+      </material>
+    </visual>
   </link>
   <joint
@@ -204,39 +165,39 @@
   </joint>
   <link
-    name="l_thigh_yaw">
-    <inertial>
-      <origin
-        xyz="-1.5406E-05 -0.039347 -0.093587"
-        rpy="0 0 0" />
-      <mass
-        value="2.72" />
-      <inertia
-        ixx="0.00754800"
-        ixy="0"
-        ixz="0"
-        iyy="0.00754800"
-        iyz="0"
-        izz="0.00489600" />
-    </inertial>
-    <visual>
-      <origin
-        xyz="0 0 0"
-        rpy="0 0 0" />
-      <geometry>
-        <mesh
-          filename="/home/wl/Documents/simulation_all_ros2/src/robot_description/gh1/meshes/L2_link.STL" />
-      </geometry>
-      <material
-        name="">
-        <color
-          rgba="1 1 1 0.3" />
-      </material>
-    </visual>
-    <collision>
-      <origin
-        xyz="0 -0.01 -0.13"
-        rpy="-1.57 0 0" />
-      <geometry>
-        <cylinder radius="0.06" length="0.15" />
+    name="l_thigh_roll">
+    <inertial>
+      <origin
+        xyz="0.078159 0.0 0.003801"
+        rpy="0 0 0" />
+      <mass
+        value="2.19" />
+      <inertia
+        ixx="0.00262800"
+        ixy="0"
+        ixz="0"
+        iyy="0.00262800"
+        iyz="0"
+        izz="0.00394200" />
+    </inertial>
+    <visual>
+      <origin
+        xyz="0 0 0"
+        rpy="0 0 0" />
+      <geometry>
+        <mesh
+          filename="/home/wl/Documents/simulation_all_ros2/src/robot_description/gh1/meshes/L1_link.STL" />
+      </geometry>
+      <material
+        name="">
+        <color
+          rgba="1 1 1 0.3" />
+      </material>
+    </visual>
+    <collision>
+      <origin
+        xyz="0.085 0 0"
+        rpy="0 0 0" />
+      <geometry>
+        <cylinder radius="0.06" length="0.06" />
       </geometry>
     </collision>
@@ -258,39 +219,40 @@
       velocity="12.552" />
   </joint>
-  <link name="l_thigh_pitch">
-    <inertial>
-      <origin
-        xyz="0.0075478 0.052643 -0.12044"
-        rpy="0 0 0" />
-      <mass
-        value="4.07" />
-      <inertia
-        ixx="0.04239583"
-        ixy="0"
-        ixz="0"
-        iyy="0.04320983"
-        iyz="0"
-        izz="0.00250983" />
-    </inertial>
-    <visual>
-      <origin
-        xyz="0 0 0"
-        rpy="0 0 0" />
-      <geometry>
-        <mesh
-          filename="/home/wl/Documents/simulation_all_ros2/src/robot_description/gh1/meshes/L3_link.STL" />
-      </geometry>
-      <material
-        name="">
-        <color
-          rgba="1 1 1 0.3" />
-      </material>
-    </visual>
-    <collision>
-      <origin
-        xyz="0.02 0.04 -0.25"
-        rpy="0 0 0" />
-      <geometry>
-        <box size="0.07 0.05 0.35"/>
+  <link
+    name="l_thigh_yaw">
+    <inertial>
+      <origin
+        xyz="-1.5406E-05 -0.039347 -0.093587"
+        rpy="0 0 0" />
+      <mass
+        value="2.72" />
+      <inertia
+        ixx="0.00754800"
+        ixy="0"
+        ixz="0"
+        iyy="0.00754800"
+        iyz="0"
+        izz="0.00489600" />
+    </inertial>
+    <visual>
+      <origin
+        xyz="0 0 0"
+        rpy="0 0 0" />
+      <geometry>
+        <mesh
+          filename="/home/wl/Documents/simulation_all_ros2/src/robot_description/gh1/meshes/L2_link.STL" />
+      </geometry>
+      <material
+        name="">
+        <color
+          rgba="1 1 1 0.3" />
+      </material>
+    </visual>
+    <collision>
+      <origin
+        xyz="0 -0.01 -0.13"
+        rpy="-1.57 0 0" />
+      <geometry>
+        <cylinder radius="0.06" length="0.15" />
       </geometry>
     </collision>
@@ -310,39 +272,39 @@
       velocity="20.92" />
   </joint>
-  <link name="l_shank_pitch">
-    <inertial>
-      <origin
-        xyz="0.0023769 -0.0025816 -0.15422"
-        rpy="0 0 0" />
-      <mass
-        value="1.88" />
-      <inertia
-        ixx="0.01617442"
-        ixy="0"
-        ixz="0"
-        iyy="0.01660667"
-        iyz="0"
-        izz="0.00069576" />
-    </inertial>
-    <visual>
-      <origin
-        xyz="0 0 0"
-        rpy="0 0 0" />
-      <geometry>
-        <mesh
-          filename="/home/wl/Documents/simulation_all_ros2/src/robot_description/gh1/meshes/L4_link.STL" />
-      </geometry>
-      <material
-        name="">
-        <color
-          rgba="1 1 1 0.3" />
-      </material>
-    </visual>
-    <collision>
-      <origin
-        xyz="0 0 -0.22"
-        rpy="0 0 0" />
-      <geometry>
-        <box size="0.06 0.029 0.32"/>
+  <link name="l_thigh_pitch">
+    <inertial>
+      <origin
+        xyz="0.0075478 0.052643 -0.12044"
+        rpy="0 0 0" />
+      <mass
+        value="4.07" />
+      <inertia
+        ixx="0.04239583"
+        ixy="0"
+        ixz="0"
+        iyy="0.04320983"
+        iyz="0"
+        izz="0.00250983" />
+    </inertial>
+    <visual>
+      <origin
+        xyz="0 0 0"
+        rpy="0 0 0" />
+      <geometry>
+        <mesh
+          filename="/home/wl/Documents/simulation_all_ros2/src/robot_description/gh1/meshes/L3_link.STL" />
+      </geometry>
+      <material
+        name="">
+        <color
+          rgba="1 1 1 0.3" />
+      </material>
+    </visual>
+    <collision>
+      <origin
+        xyz="0.02 0.04 -0.25"
+        rpy="0 0 0" />
+      <geometry>
+        <box size="0.07 0.05 0.35"/>
       </geometry>
     </collision>
@@ -362,63 +324,39 @@
       velocity="20.92" />
   </joint>
-  <link name="l_foot_pitch">
-    <inertial>
-      <origin
-        xyz="0.022131 0.0001084 -0.040348"
-        rpy="0 0 0" />
-      <mass
-        value="0.55" />
-      <inertia
-        ixx="0.00013292"
-        ixy="0"
-        ixz="0"
-        iyy="0.00288292"
-        iyz="0"
-        izz="0.00297917" />
-    </inertial>
-    <visual>
-      <origin
-        xyz="0 0 0"
-        rpy="0 0 0" />
-      <geometry>
-        <mesh
-          filename="/home/wl/Documents/simulation_all_ros2/src/robot_description/gh1/meshes/L5_link.STL" />
-      </geometry>
-      <material
-        name="">
-        <color
-          rgba="1 1 1 0.3" />
-      </material>
-    </visual>
-    <!-- <collision>
-      <origin
-        xyz="0.025 0 -0.045"
-        rpy="0 0 0" />
-      <geometry>
-        <box size="0.25 0.05 0.02"/>
-      </geometry>
-    </collision> -->
-    <collision>
-      <origin
-        xyz="0.02 0 -0.04"
-        rpy="0 1.57 0" />
-      <geometry>
-        <cylinder radius="0.015" length="0.22"/>
-      </geometry>
-    </collision>
-    <collision>
-      <origin
-        xyz="0.13 0 -0.04"
-        rpy="0 0 0" />
-      <geometry>
-        <sphere radius="0.015"/>
-      </geometry>
-    </collision>
-    <collision>
-      <origin
-        xyz="-0.09 0 -0.04"
-        rpy="0 0 0" />
-      <geometry>
-        <sphere radius="0.015"/>
+  <link name="l_shank_pitch">
+    <inertial>
+      <origin
+        xyz="0.0023769 -0.0025816 -0.15422"
+        rpy="0 0 0" />
+      <mass
+        value="1.88" />
+      <inertia
+        ixx="0.01617442"
+        ixy="0"
+        ixz="0"
+        iyy="0.01660667"
+        iyz="0"
+        izz="0.00069576" />
+    </inertial>
+    <visual>
+      <origin
+        xyz="0 0 0"
+        rpy="0 0 0" />
+      <geometry>
+        <mesh
+          filename="/home/wl/Documents/simulation_all_ros2/src/robot_description/gh1/meshes/L4_link.STL" />
+      </geometry>
+      <material
+        name="">
+        <color
+          rgba="1 1 1 0.3" />
+      </material>
+    </visual>
+    <collision>
+      <origin
+        xyz="0 0 -0.22"
+        rpy="0 0 0" />
+      <geometry>
+        <box size="0.06 0.029 0.32"/>
       </geometry>
     </collision>
@@ -438,4 +376,66 @@
       velocity="46.024" />
   </joint>
+  <link name="l_foot_pitch">
+    <inertial>
+      <origin
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