Commit message: 将mz\sz\iris的description等描述文件按照gh1的格式移植完成,给iris配置ros2自带的joint_trajectory_controller控制器,配置的command_interface类型为position,并且没有effort仅有acceleration state_interface返回

File: src/robot_description/gh1/xacro/robot_description.xacro (robot description, xacro)
@@ -1,5 +1,5 @@
 <?xml version="1.0"?>
 <robot xmlns:xacro="http://www.ros.org/wiki/xacro">
-    <xacro:macro name="gh1" params="debug">
+    <xacro:macro name="gh1_description" params="debug">
     <!-- Rotor related joint and link is only for demonstrate location. -->
     <!-- Actually, the rotor will rotate and the joint is not fixed. Reduction ratio should be

File: src/robot_description/gh1/xacro/robot_system.xacro (robot description, xacro)
@@ -6,4 +6,4 @@
   <xacro:include filename="$(find gh1)/xacro/ros2_control.xacro" />
   <xacro:gh1_ros2_control/>
-  <xacro:gh1 debug="$(arg debug)"/>
+  <xacro:gh1_description debug="$(arg debug)"/>
 </robot>
